File: hardware/branch_v1/branch_v1.kicad_sch (KiCad schematic)
At the start: 88 parts, among them J1 BUS_IN 2x20, J10 STRAND0, J11 STRAND1, J12 STRAND2, J13 STRAND3, J14 STRAND4, J15 STRAND5, J16 STRAND6, J17 STRAND7, J18 STRAND8, J19 STRAND9, J2 BUS_OUT 2x20, J20 STRAND10, J21 STRAND11, J22 STRAND12, J23 STRAND13, J24 STRAND14, J25 STRAND15, J30 5V_INJECT, J31 5V_INJECT, U1 74AHCT245PW, U2 74AHCT245PW, U3 74AHCT245PW, U4 74HC688D, U5 SN74AHC1G32DBVR, U6 74AHCT245PW, U7 74AHCT245PW, U8 74AHCT245PW, U9 74AHCT245PW

Commit message: v1.1: 12V distribution + eFuse/buck/PTC/ESD on branch; main board layout DRC 0 (structured spine routing, arcs), 12V input chain, fab outputs, renders, LAYOUT_LESSONS
Parts:
- removed C1, C2, C3, C4, C5, C6, C7, C8, C9: 100nF, Capacitor_SMD:C_0603_1608Metric, symbol cube:100nF_2__91474
- removed C10, C11, C12, C13, C14, C15: 47uF, Capacitor_SMD:C_0805_2012Metric, symbol cube:47uF_2__91474
- removed J1: BUS_IN 2x20, Connector_IDC:IDC-Header_2x20_P2.54mm_Vertical, symbol cube:BUS_IN_2x20_40__97826
- removed J10: STRAND0, Connector_JST:JST_XH_B4B-XH-A_1x04_P2.50mm_Vertical, symbol cube:STRAND0_4__13197
- removed J11: STRAND1, Connector_JST:JST_XH_B4B-XH-A_1x04_P2.50mm_Vertical, symbol cube:STRAND1_4__13197
- removed J12: STRAND2, Connector_JST:JST_XH_B4B-XH-A_1x04_P2.50mm_Vertical, symbol cube:STRAND2_4__13197
- removed J13: STRAND3, Connector_JST:JST_XH_B4B-XH-A_1x04_P2.50mm_Vertical, symbol cube:STRAND3_4__13197
- removed J14: STRAND4, Connector_JST:JST_XH_B4B-XH-A_1x04_P2.50mm_Vertical, symbol cube:STRAND4_4__13197
- removed J15: STRAND5, Connector_JST:JST_XH_B4B-XH-A_1x04_P2.50mm_Vertical, symbol cube:STRAND5_4__13197
- removed J16: STRAND6, Connector_JST:JST_XH_B4B-XH-A_1x04_P2.50mm_Vertical, symbol cube:STRAND6_4__13197
- removed J17: STRAND7, Connector_JST:JST_XH_B4B-XH-A_1x04_P2.50mm_Vertical, symbol cube:STRAND7_4__13197
- removed J18: STRAND8, Connector_JST:JST_XH_B4B-XH-A_1x04_P2.50mm_Vertical, symbol cube:STRAND8_4__13197
- removed J19: STRAND9, Connector_JST:JST_XH_B4B-XH-A_1x04_P2.50mm_Vertical, symbol cube:STRAND9_4__13197
- removed J2: BUS_OUT 2x20, Connector_IDC:IDC-Header_2x20_P2.54mm_Vertical, symbol cube:BUS_OUT_2x20_40__97826
- removed J20: STRAND10, Connector_JST:JST_XH_B4B-XH-A_1x04_P2.50mm_Vertical, symbol cube:STRAND10_4__13197
- removed J21: STRAND11, Connector_JST:JST_XH_B4B-XH-A_1x04_P2.50mm_Vertical, symbol cube:STRAND11_4__13197
- removed J22: STRAND12, Connector_JST:JST_XH_B4B-XH-A_1x04_P2.50mm_Vertical, symbol cube:STRAND12_4__13197
- removed J23: STRAND13, Connector_JST:JST_XH_B4B-XH-A_1x04_P2.50mm_Vertical, symbol cube:STRAND13_4__13197
- removed J24: STRAND14, Connector_JST:JST_XH_B4B-XH-A_1x04_P2.50mm_Vertical, symbol cube:STRAND14_4__13197
- removed J25: STRAND15, Connector_JST:JST_XH_B4B-XH-A_1x04_P2.50mm_Vertical, symbol cube:STRAND15_4__13197
- removed J30, J31: 5V_INJECT, TerminalBlock_Phoenix:TerminalBlock_Phoenix_MKDS-1,5-2-5.08_1x02_P5.08mm_Horizontal, symbol cube:5V_INJECT_2__14566
- removed JP0: ID0_SET, Jumper:SolderJumper-2_P1.3mm_Open_RoundedPad1.0x1.5mm, symbol cube:ID0_SET_2__91474
- removed JP1: ID1_SET, Jumper:SolderJumper-2_P1.3mm_Open_RoundedPad1.0x1.5mm, symbol cube:ID1_SET_2__91474
- removed JP2: ID2_SET, Jumper:SolderJumper-2_P1.3mm_Open_RoundedPad1.0x1.5mm, symbol cube:ID2_SET_2__91474
- removed JP3: ID3_SET, Jumper:SolderJumper-2_P1.3mm_Open_RoundedPad1.0x1.5mm, symbol cube:ID3_SET_2__91474
- removed JP4: ID4_SET, Jumper:SolderJumper-2_P1.3mm_Open_RoundedPad1.0x1.5mm, symbol cube:ID4_SET_2__91474
- removed JP5: ID5_SET, Jumper:SolderJumper-2_P1.3mm_Open_RoundedPad1.0x1.5mm, symbol cube:ID5_SET_2__91474
- removed RC0, RC1, RC10, RC11, RC12, RC13, RC14, RC15, RC2, RC3, RC4, RC5, RC6, RC7, RC8, RC9, RD0, RD1, RD10, RD11, RD12, RD13, RD14, RD15, RD2, RD3, RD4, RD5, RD6, RD7, RD8, RD9: 33R, Resistor_SMD:R_0603_1608Metric, symbol cube:33R_2__91474
- removed RID0, RID1, RID2, RID3, RID4, RID5: 10k, Resistor_SMD:R_0603_1608Metric, symbol cube:10k_2__91474
- removed U1, U2, U3, U6, U7, U8, U9: 74AHCT245PW, Package_SO:TSSOP-20_4.4x6.5mm_P0.65mm, symbol cube:74AHCT245PW_20__84077
- removed U4: 74HC688D, Package_SO:SOIC-20W_7.5x12.8mm_P1.27mm, symbol cube:74HC688D_20__31776
- removed U5: SN74AHC1G32DBVR, Package_TO_SOT_SMD:SOT-23-5, symbol cube:SN74AHC1G32DBVR_5__37443
- added C1, C2, C3, C36, C4, C5, C6, C7, C8, C9: 100nF, Capacitor_SMD:C_0603_1608Metric, symbol cube:100nF_2__21234
- added C10, C11, C12, C13, C14, C15: 47uF, Capacitor_SMD:C_0805_2012Metric, symbol cube:47uF_2__21234
- added C30, C31: 10nF, Capacitor_SMD:C_0603_1608Metric, symbol cube:10nF_2__21234
- added C32, C33, C34, C35: 10uF/50V, Capacitor_SMD:C_1206_3216Metric, symbol cube:10uF/50V_2__21234
- added C37: 4.7uF, Capacitor_SMD:C_0603_1608Metric, symbol cube:4.7uF_2__21234
- added C38: 22nF, Capacitor_SMD:C_0603_1608Metric, symbol cube:22nF_2__21234
- added C40, C41, C42, C43, C44, C45: 47uF/16V, Capacitor_SMD:C_1210_3225Metric, symbol cube:47uF/16V_2__21234
- added D30: SMBJ15A, Diode_SMD:D_SMB, symbol cube:SMBJ15A_2__46460
- added F10, F11, F12, F13, F14, F15, F16, F17, F18, F19, F20, F21, F22, F23, F24, F25: PTC 2A, Fuse:Fuse_1812_4532Metric, symbol cube:PTC_2A_2__21234
- added J1: BUS_IN 2x20, Connector_IDC:IDC-Header_2x20_P2.54mm_Vertical, symbol cube:BUS_IN_2x20_40__84700
- added J10: STRAND0, Connector_JST:JST_XH_B4B-XH-A_1x04_P2.50mm_Vertical, symbol cube:STRAND0_4__75938
- added J11: STRAND1, Connector_JST:JST_XH_B4B-XH-A_1x04_P2.50mm_Vertical, symbol cube:STRAND1_4__75938
- added J12: STRAND2, Connector_JST:JST_XH_B4B-XH-A_1x04_P2.50mm_Vertical, symbol cube:STRAND2_4__75938
- added J13: STRAND3, Connector_JST:JST_XH_B4B-XH-A_1x04_P2.50mm_Vertical, symbol cube:STRAND3_4__75938
- added J14: STRAND4, Connector_JST:JST_XH_B4B-XH-A_1x04_P2.50mm_Vertical, symbol cube:STRAND4_4__75938
- added J15: STRAND5, Connector_JST:JST_XH_B4B-XH-A_1x04_P2.50mm_Vertical, symbol cube:STRAND5_4__75938
- added J16: STRAND6, Connector_JST:JST_XH_B4B-XH-A_1x04_P2.50mm_Vertical, symbol cube:STRAND6_4__75938
- added J17: STRAND7, Connector_JST:JST_XH_B4B-XH-A_1x04_P2.50mm_Vertical, symbol cube:STRAND7_4__75938
- added J18: STRAND8, Connector_JST:JST_XH_B4B-XH-A_1x04_P2.50mm_Vertical, symbol cube:STRAND8_4__75938
- added J19: STRAND9, Connector_JST:JST_XH_B4B-XH-A_1x04_P2.50mm_Vertical, symbol cube:STRAND9_4__75938
- added J2: BUS_OUT 2x20, Connector_IDC:IDC-Header_2x20_P2.54mm_Vertical, symbol cube:BUS_OUT_2x20_40__84700
- added J20: STRAND10, Connector_JST:JST_XH_B4B-XH-A_1x04_P2.50mm_Vertical, symbol cube:STRAND10_4__75938
- added J21: STRAND11, Connector_JST:JST_XH_B4B-XH-A_1x04_P2.50mm_Vertical, symbol cube:STRAND11_4__75938
- added J22: STRAND12, Connector_JST:JST_XH_B4B-XH-A_1x04_P2.50mm_Vertical, symbol cube:STRAND12_4__75938
- added J23: STRAND13, Connector_JST:JST_XH_B4B-XH-A_1x04_P2.50mm_Vertical, symbol cube:STRAND13_4__75938
- added J24: STRAND14, Connector_JST:JST_XH_B4B-XH-A_1x04_P2.50mm_Vertical, symbol cube:STRAND14_4__75938
- added J25: STRAND15, Connector_JST:JST_XH_B4B-XH-A_1x04_P2.50mm_Vertical, symbol cube:STRAND15_4__75938
- added J30, J31: 12V_BUS, TerminalBlock_Phoenix:TerminalBlock_Phoenix_MKDS-1,5-2-5.08_1x02_P5.08mm_Horizontal, symbol cube:12V_BUS_2__37452
- added JP0: ID0_SET, Jumper:SolderJumper-2_P1.3mm_Open_RoundedPad1.0x1.5mm, symbol cube:ID0_SET_2__21234
- added JP1: ID1_SET, Jumper:SolderJumper-2_P1.3mm_Open_RoundedPad1.0x1.5mm, symbol cube:ID1_SET_2__21234
- added JP2: ID2_SET, Jumper:SolderJumper-2_P1.3mm_Open_RoundedPad1.0x1.5mm, symbol cube:ID2_SET_2__21234
- added JP3: ID3_SET, Jumper:SolderJumper-2_P1.3mm_Open_RoundedPad1.0x1.5mm, symbol cube:ID3_SET_2__21234
- added JP4: ID4_SET, Jumper:SolderJumper-2_P1.3mm_Open_RoundedPad1.0x1.5mm, symbol cube:ID4_SET_2__21234
- added JP5: ID5_SET, Jumper:SolderJumper-2_P1.3mm_Open_RoundedPad1.0x1.5mm, symbol cube:ID5_SET_2__21234
- added L30: 1.5uH 20A, Inductor_SMD:L_TaiTech_TMPC1265_13.5x12.5mm, symbol cube:1.5uH_20A_2__21234
- added R30, R40: 100k, Resistor_SMD:R_0603_1608Metric, symbol cube:100k_2__21234
- added R31: 15k, Resistor_SMD:R_0603_1608Metric, symbol cube:15k_2__21234
- added R32: 8.2k, Resistor_SMD:R_0603_1608Metric, symbol cube:8.2k_2__21234
- added R33: 750R, Resistor_SMD:R_0603_1608Metric, symbol cube:750R_2__21234
- added R34, R36, R39, RID0, RID1, RID2, RID3, RID4, RID5: 10k, Resistor_SMD:R_0603_1608Metric, symbol cube:10k_2__21234
- added R35: 75k, Resistor_SMD:R_0603_1608Metric, symbol cube:75k_2__21234
- added R37: 120k, Resistor_SMD:R_0603_1608Metric, symbol cube:120k_2__21234
- added R38: 20k, Resistor_SMD:R_0603_1608Metric, symbol cube:20k_2__21234
- added RC0, RC1, RC10, RC11, RC12, RC13, RC14, RC15, RC2, RC3, RC4, RC5, RC6, RC7, RC8, RC9, RD0, RD1, RD10, RD11, RD12, RD13, RD14, RD15, RD2, RD3, RD4, RD5, RD6, RD7, RD8, RD9: 33R, Resistor_SMD:R_0603_1608Metric, symbol cube:33R_2__21234
- added U1, U2, U3, U6, U7, U8, U9: 74AHCT245PW, Package_SO:TSSOP-20_4.4x6.5mm_P0.65mm, symbol cube:74AHCT245PW_20__32821
- added U30: TPS259474LRPWR, cube:TI_RPW0010A_VQFN-HR-10_2x2mm_P0.45mm, symbol cube:TPS259474LRPWR_10__27248
- added U31: TPS56C215RNNR, Package_DFN_QFN:Texas_RNN0018A, symbol cube:TPS56C215RNNR_18__22882
- added U4: 74HC688D, Package_SO:SOIC-20W_7.5x12.8mm_P1.27mm, symbol cube:74HC688D_20__12603
- added U5: SN74AHC1G32DBVR, Package_TO_SOT_SMD:SOT-23-5, symbol cube:SN74AHC1G32DBVR_5__15265
- added UE0, UE1, UE10, UE11, UE12, UE13, UE14, UE15, UE2, UE3, UE4, UE5, UE6, UE7, UE8, UE9: USBLC6-2SC6, Package_TO_SOT_SMD:SOT-23-6, symbol cube:USBLC6-2SC6_6__29574
Connections:
- net +5V: now also C1.1, C10.1, C11.1, C12.1, C13.1, C14.1, C15.1, C2.1, C3.1, C4.1, C40.1, C41.1, C42.1, C43.1, C44.1, C45.1, C5.1, C6.1, C7.1, C8.1, C9.1, F10.1, F11.1, F12.1, F13.1, F14.1, F15.1, F16.1, F17.1, F18.1, F19.1, F20.1, F21.1, F22.1, F23.1, F24.1, F25.1, L30.2, R34.2, R35.1, R39.2, RID0.1, RID1.1, RID2.1, RID3.1, RID4.1, RID5.1, U1.1 (DIR), U1.20 (VCC), U2.1 (DIR), U2.20 (VCC), U3.1 (DIR), U3.20 (VCC), U4.20 (VCC), U5.5 (VCC), U6.1 (DIR), U6.20 (VCC), U7.1 (DIR), U7.20 (VCC), U8.1 (DIR), U8.20 (VCC), U9.1 (DIR), U9.20 (VCC), UE0.5 (VBUS), UE1.5 (VBUS), UE10.5 (VBUS), UE11.5 (VBUS), UE12.5 (VBUS), UE13.5 (VBUS), UE14.5 (VBUS), UE15.5 (VBUS), UE2.5 (VBUS), UE3.5 (VBUS), UE4.5 (VBUS), UE5.5 (VBUS), UE6.5 (VBUS), UE7.5 (VBUS), UE8.5 (VBUS), UE9.5 (VBUS)
- net GCLK: now also U5.4 (Y), U8.2 (A1), U8.3 (A2), U8.4 (A3), U8.5 (A4), U8.6 (A5), U8.7 (A6), U8.8 (A7), U8.9 (A8), U9.2 (A1), U9.3 (A2), U9.4 (A3), U9.5 (A4), U9.6 (A5), U9.7 (A6), U9.8 (A7), U9.9 (A8)
- net GND: now also C1.2, C10.2, C11.2, C12.2, C13.2, C14.2, C15.2, C2.2, C3.2, C30.2, C31.2, C32.2, C33.2, C34.2, C35.2, C37.2, C38.2, C4.2, C40.2, C41.2, C42.2, C43.2, C44.2, C45.2, C5.2, C6.2, C7.2, C8.2, C9.2, D30.2 (A), J1.10 (GND), J1.12 (GND), J1.14 (GND), J1.16 (GND), J1.18 (GND), J1.2 (GND), J1.20 (GND), J1.22 (GND), J1.24 (GND), J1.26 (GND), J1.28 (GND), J1.30 (GND), J1.32 (GND), J1.4 (GND), J1.40 (GND), J1.6 (GND), J1.8 (GND), J10.4 (GND), J11.4 (GND), J12.4 (GND), J13.4 (GND), J14.4 (GND), J15.4 (GND), J16.4 (GND), J17.4 (GND), J18.4 (GND), J19.4 (GND), J2.10 (GND), J2.12 (GND), J2.14 (GND), J2.16 (GND), J2.18 (GND), J2.2 (GND), J2.20 (GND), J2.22 (GND), J2.24 (GND), J2.26 (GND), J2.28 (GND), J2.30 (GND), J2.32 (GND), J2.4 (GND), J2.40 (GND), J2.6 (GND), J2.8 (GND), J20.4 (GND), J21.4 (GND), J22.4 (GND), J23.4 (GND), J24.4 (GND), J25.4 (GND), J30.2 (GND), J31.2 (GND), JP0.2, JP1.2, JP2.2, JP3.2, JP4.2, JP5.2, R31.2, R32.2, R33.2, R36.2, R38.2, U1.10 (GND), U1.19 (~OE), U2.10 (GND), U2.19 (~OE), U3.10 (GND), U3.19 (~OE), U3.9 (A8), U30.8 (GND), U31.10 (PGND_6), U31.12 (AGND), U31.3 (PGND), U31.4 (PGND_2), U31.5 (PGND_3), U31.8 (PGND_4), U31.9 (PGND_5), U4.1 (~G), U4.10 (GND), U4.15 (P6), U4.16 (Q6), U4.17 (P7), U4.18 (Q7), U5.3 (GND), U6.10 (GND), U6.19 (~OE), U7.10 (GND), U7.19 (~OE), U8.10 (GND), U8.19 (~OE), U9.10 (GND), U9.19 (~OE), UE0.2 (GND), UE1.2 (GND), UE10.2 (GND), UE11.2 (GND), UE12.2 (GND), UE13.2 (GND), UE14.2 (GND), UE15.2 (GND), UE2.2 (GND), UE3.2 (GND), UE4.2 (GND), UE5.2 (GND), UE6.2 (GND), UE7.2 (GND), UE8.2 (GND), UE9.2 (GND)
- net ID0: now also JP0.1, RID0.2, U4.3 (Q0)
- net ID1: now also JP1.1, RID1.2, U4.5 (Q1)
- net ID2: now also JP2.1, RID2.2, U4.7 (Q2)
- net ID3: now also JP3.1, RID3.2, U4.9 (Q3)
- net ID4: now also JP4.1, RID4.2, U4.12 (Q4)
- net ID5: now also JP5.1, RID5.2, U4.14 (Q5)
- net IN_A0: now also J1.35 (A0), U3.3 (A2)
- net IN_A1: now also J1.37 (A1), U3.4 (A3)
- net IN_A2: now also J1.39 (A2), U3.5 (A4)
- net IN_A3: now also J1.34 (A3), U3.6 (A5)
- net IN_A4: now also J1.36 (A4), U3.7 (A6)
- net IN_A5: now also J1.38 (A5), U3.8 (A7)
- net IN_CLK: now also J1.33 (CLK), U3.2 (A1)
- net IN_D0: now also J1.1 (D0), U1.2 (A1)
- net IN_D1: now also J1.3 (D1), U1.3 (A2)
- net IN_D10: now also J1.21 (D10), U2.4 (A3)
- net IN_D11: now also J1.23 (D11), U2.5 (A4)
- net IN_D12: now also J1.25 (D12), U2.6 (A5)
- net IN_D13: now also J1.27 (D13), U2.7 (A6)
- net IN_D14: now also J1.29 (D14), U2.8 (A7)
- net IN_D15: now also J1.31 (D15), U2.9 (A8)
- net IN_D2: now also J1.5 (D2), U1.4 (A3)
- net IN_D3: now also J1.7 (D3), U1.5 (A4)
- net IN_D4: now also J1.9 (D4), U1.6 (A5)
- net IN_D5: now also J1.11 (D5), U1.7 (A6)
- net IN_D6: now also J1.13 (D6), U1.8 (A7)
- net IN_D7: now also J1.15 (D7), U1.9 (A8)
- net IN_D8: now also J1.17 (D8), U2.2 (A1)
- net IN_D9: now also J1.19 (D9), U2.3 (A2)
- net L_A0: now also J2.35 (A0), U3.17 (B2), U4.2 (P0)
- net L_A1: now also J2.37 (A1), U3.16 (B3), U4.4 (P1)
- net L_A2: now also J2.39 (A2), U3.15 (B4), U4.6 (P2)
- net L_A3: now also J2.34 (A3), U3.14 (B5), U4.8 (P3)
- net L_A4: now also J2.36 (A4), U3.13 (B6), U4.11 (P4)
- net L_A5: now also J2.38 (A5), U3.12 (B7), U4.13 (P5)
- net L_CLK: now also J2.33 (CLK), U3.18 (B1), U5.1 (A)
- net L_D0: now also J2.1 (D0), U1.18 (B1), U6.2 (A1)
- net L_D1: now also J2.3 (D1), U1.17 (B2), U6.3 (A2)
- net L_D10: now also J2.21 (D10), U2.16 (B3), U7.4 (A3)
- net L_D11: now also J2.23 (D11), U2.15 (B4), U7.5 (A4)
- net L_D12: now also J2.25 (D12), U2.14 (B5), U7.6 (A5)
- net L_D13: now also J2.27 (D13), U2.13 (B6), U7.7 (A6)
- net L_D14: now also J2.29 (D14), U2.12 (B7), U7.8 (A7)
- net L_D15: now also J2.31 (D15), U2.11 (B8), U7.9 (A8)
- net L_D2: now also J2.5 (D2), U1.16 (B3), U6.4 (A3)
- net L_D3: now also J2.7 (D3), U1.15 (B4), U6.5 (A4)
- net L_D4: now also J2.9 (D4), U1.14 (B5), U6.6 (A5)
- net L_D5: now also J2.11 (D5), U1.13 (B6), U6.7 (A6)
- net L_D6: now also J2.13 (D6), U1.12 (B7), U6.8 (A7)
- net L_D7: now also J2.15 (D7), U1.11 (B8), U6.9 (A8)
- net L_D8: now also J2.17 (D8), U2.18 (B1), U7.2 (A1)
- net L_D9: now also J2.19 (D9), U2.17 (B2), U7.3 (A2)
- net SC0: now also J10.3 (CLK), RC0.2, UE0.3 (IO2), UE0.4 (IO2b)
- net SC1: now also J11.3 (CLK), RC1.2, UE1.3 (IO2), UE1.4 (IO2b)
- net SC10: now also J20.3 (CLK), RC10.2, UE10.3 (IO2), UE10.4 (IO2b)
- net SC11: now also J21.3 (CLK), RC11.2, UE11.3 (IO2), UE11.4 (IO2b)
- net SC12: now also J22.3 (CLK), RC12.2, UE12.3 (IO2), UE12.4 (IO2b)
- net SC13: now also J23.3 (CLK), RC13.2, UE13.3 (IO2), UE13.4 (IO2b)
- net SC14: now also J24.3 (CLK), RC14.2, UE14.3 (IO2), UE14.4 (IO2b)
- net SC15: now also J25.3 (CLK), RC15.2, UE15.3 (IO2), UE15.4 (IO2b)
- net SC2: now also J12.3 (CLK), RC2.2, UE2.3 (IO2), UE2.4 (IO2b)
- net SC3: now also J13.3 (CLK), RC3.2, UE3.3 (IO2), UE3.4 (IO2b)
- net SC4: now also J14.3 (CLK), RC4.2, UE4.3 (IO2), UE4.4 (IO2b)
- net SC5: now also J15.3 (CLK), RC5.2, UE5.3 (IO2), UE5.4 (IO2b)
- net SC6: now also J16.3 (CLK), RC6.2, UE6.3 (IO2), UE6.4 (IO2b)
- net SC7: now also J17.3 (CLK), RC7.2, UE7.3 (IO2), UE7.4 (IO2b)
- net SC8: now also J18.3 (CLK), RC8.2, UE8.3 (IO2), UE8.4 (IO2b)
- net SC9: now also J19.3 (CLK), RC9.2, UE9.3 (IO2), UE9.4 (IO2b)
- net SCR0: now also RC0.1, U8.18 (B1)
- net SCR1: now also RC1.1, U8.17 (B2)
- net SCR10: now also RC10.1, U9.16 (B3)
- net SCR11: now also RC11.1, U9.15 (B4)
- net SCR12: now also RC12.1, U9.14 (B5)
- net SCR13: now also RC13.1, U9.13 (B6)
- net SCR14: now also RC14.1, U9.12 (B7)
- net SCR15: now also RC15.1, U9.11 (B8)
- net SCR2: now also RC2.1, U8.16 (B3)
- net SCR3: now also RC3.1, U8.15 (B4)
- net SCR4: now also RC4.1, U8.14 (B5)
- net SCR5: now also RC5.1, U8.13 (B6)
- net SCR6: now also RC6.1, U8.12 (B7)
- net SCR7: now also RC7.1, U8.11 (B8)
- net SCR8: now also RC8.1, U9.18 (B1)
- net SCR9: now also RC9.1, U9.17 (B2)
- net SD0: now also J10.2 (DATA), RD0.2, UE0.1 (IO1), UE0.6 (IO1b)
- net SD1: now also J11.2 (DATA), RD1.2, UE1.1 (IO1), UE1.6 (IO1b)
- net SD10: now also J20.2 (DATA), RD10.2, UE10.1 (IO1), UE10.6 (IO1b)
- net SD11: now also J21.2 (DATA), RD11.2, UE11.1 (IO1), UE11.6 (IO1b)
- net SD12: now also J22.2 (DATA), RD12.2, UE12.1 (IO1), UE12.6 (IO1b)
- net SD13: now also J23.2 (DATA), RD13.2, UE13.1 (IO1), UE13.6 (IO1b)
- net SD14: now also J24.2 (DATA), RD14.2, UE14.1 (IO1), UE14.6 (IO1b)
- net SD15: now also J25.2 (DATA), RD15.2, UE15.1 (IO1), UE15.6 (IO1b)
- net SD2: now also J12.2 (DATA), RD2.2, UE2.1 (IO1), UE2.6 (IO1b)
- net SD3: now also J13.2 (DATA), RD3.2, UE3.1 (IO1), UE3.6 (IO1b)
- net SD4: now also J14.2 (DATA), RD4.2, UE4.1 (IO1), UE4.6 (IO1b)
- net SD5: now also J15.2 (DATA), RD5.2, UE5.1 (IO1), UE5.6 (IO1b)
- net SD6: now also J16.2 (DATA), RD6.2, UE6.1 (IO1), UE6.6 (IO1b)
- net SD7: now also J17.2 (DATA), RD7.2, UE7.1 (IO1), UE7.6 (IO1b)
- net SD8: now also J18.2 (DATA), RD8.2, UE8.1 (IO1), UE8.6 (IO1b)
- net SD9: now also J19.2 (DATA), RD9.2, UE9.1 (IO1), UE9.6 (IO1b)
- net SDR0: now also RD0.1, U6.18 (B1)
- net SDR1: now also RD1.1, U6.17 (B2)
- net SDR10: now also RD10.1, U7.16 (B3)
- net SDR11: now also RD11.1, U7.15 (B4)
- net SDR12: now also RD12.1, U7.14 (B5)
- net SDR13: now also RD13.1, U7.13 (B6)
- net SDR14: now also RD14.1, U7.12 (B7)
- net SDR15: now also RD15.1, U7.11 (B8)
- net SDR2: now also RD2.1, U6.16 (B3)
- net SDR3: now also RD3.1, U6.15 (B4)
- net SDR4: now also RD4.1, U6.14 (B5)
- net SDR5: now also RD5.1, U6.13 (B6)
- net SDR6: now also RD6.1, U6.12 (B7)
- net SDR7: now also RD7.1, U6.11 (B8)
- net SDR8: now also RD8.1, U7.18 (B1)
- net SDR9: now also RD9.1, U7.17 (B2)
- net SEL_N: now also U4.19 (~P=Q), U5.2 (B)
- new net +12V: C33.1, C34.1, C35.1, U30.6 (OUT), U31.11 (VIN_2), U31.15 (EN), U31.2 (VIN)
- new net BST: C36.1, U31.1 (BOOT)
- new net DVDT: C30.1, U30.7 (DVDT)
- new net EFEN: R30.2, R31.1, U30.1 (EN/UVLO), U30.4 (PGTH)
- new net EFOV: R32.1, R40.2, U30.2 (OVLO)
- new net FB5: R35.2, R36.1, U31.13 (FB)
- new net ILM: R33.1, U30.9 (ILM)
- new net ITMR: C31.1, U30.10 (ITIMER)
- new net MODE5: R37.2, R38.1, U31.18 (MODE)
- new net PG12: R34.1, U30.3 (PG)
- new net PG5: R39.1, U31.16 (PGOOD)
- new net SS5: C38.1, U31.14 (SS)
- new net SW5: C36.2, L30.1, U31.6 (SW), U31.7 (SW_2)
- new net V12_IN: C32.1, D30.1 (K), J30.1 (+12V), J31.1 (+12V), R30.1, R40.1, U30.5 (IN)
- new net V5S0: F10.2, J10.1 (+5V)
- new net V5S1: F11.2, J11.1 (+5V)
- new net V5S10: F20.2, J20.1 (+5V)
- new net V5S11: F21.2, J21.1 (+5V)
- new net V5S12: F22.2, J22.1 (+5V)
- new net V5S13: F23.2, J23.1 (+5V)
- new net V5S14: F24.2, J24.1 (+5V)
- new net V5S15: F25.2, J25.1 (+5V)
- new net V5S2: F12.2, J12.1 (+5V)
- new net V5S3: F13.2, J13.1 (+5V)
- new net V5S4: F14.2, J14.1 (+5V)
- new net V5S5: F15.2, J15.1 (+5V)
- new net V5S6: F16.2, J16.1 (+5V)
- new net V5S7: F17.2, J17.1 (+5V)
- new net V5S8: F18.2, J18.1 (+5V)
- new net V5S9: F19.2, J19.1 (+5V)
- new net VREG5: C37.1, R37.1, U31.17 (VREG5)

Commit message: Size table + pixel choice, cube footprint lib (TPS25947 RPW, verified inductors), schematic->PCB linking (main parity 0), TPD4E05U06 port ESD, branch layout WIP
Parts:
- removed C1, C2, C3, C36, C4, C5, C6, C7, C8, C9: 100nF, Capacitor_SMD:C_0603_1608Metric, symbol cube:100nF_2__21234
- removed C10, C11, C12, C13, C14, C15: 47uF, Capacitor_SMD:C_0805_2012Metric, symbol cube:47uF_2__21234
- removed C30, C31: 10nF, Capacitor_SMD:C_0603_1608Metric, symbol cube:10nF_2__21234
- removed C32, C33, C34, C35: 10uF/50V, Capacitor_SMD:C_1206_3216Metric, symbol cube:10uF/50V_2__21234
- removed C37: 4.7uF, Capacitor_SMD:C_0603_1608Metric, symbol cube:4.7uF_2__21234
- removed C38: 22nF, Capacitor_SMD:C_0603_1608Metric, symbol cube:22nF_2__21234
- removed C40, C41, C42, C43, C44, C45: 47uF/16V, Capacitor_SMD:C_1210_3225Metric, symbol cube:47uF/16V_2__21234
- removed D30: SMBJ15A, Diode_SMD:D_SMB, symbol cube:SMBJ15A_2__46460
- removed F10, F11, F12, F13, F14, F15, F16, F17, F18, F19, F20, F21, F22, F23, F24, F25: PTC 2A, Fuse:Fuse_1812_4532Metric, symbol cube:PTC_2A_2__21234
- removed J1: BUS_IN 2x20, Connector_IDC:IDC-Header_2x20_P2.54mm_Vertical, symbol cube:BUS_IN_2x20_40__84700
- removed J10: STRAND0, Connector_JST:JST_XH_B4B-XH-A_1x04_P2.50mm_Vertical, symbol cube:STRAND0_4__75938
- removed J11: STRAND1, Connector_JST:JST_XH_B4B-XH-A_1x04_P2.50mm_Vertical, symbol cube:STRAND1_4__75938
- removed J12: STRAND2, Connector_JST:JST_XH_B4B-XH-A_1x04_P2.50mm_Vertical, symbol cube:STRAND2_4__75938
- removed J13: STRAND3, Connector_JST:JST_XH_B4B-XH-A_1x04_P2.50mm_Vertical, symbol cube:STRAND3_4__75938
- removed J14: STRAND4, Connector_JST:JST_XH_B4B-XH-A_1x04_P2.50mm_Vertical, symbol cube:STRAND4_4__75938
- removed J15: STRAND5, Connector_JST:JST_XH_B4B-XH-A_1x04_P2.50mm_Vertical, symbol cube:STRAND5_4__75938
- removed J16: STRAND6, Connector_JST:JST_XH_B4B-XH-A_1x04_P2.50mm_Vertical, symbol cube:STRAND6_4__75938
- removed J17: STRAND7, Connector_JST:JST_XH_B4B-XH-A_1x04_P2.50mm_Vertical, symbol cube:STRAND7_4__75938
- removed J18: STRAND8, Connector_JST:JST_XH_B4B-XH-A_1x04_P2.50mm_Vertical, symbol cube:STRAND8_4__75938
- removed J19: STRAND9, Connector_JST:JST_XH_B4B-XH-A_1x04_P2.50mm_Vertical, symbol cube:STRAND9_4__75938
- removed J2: BUS_OUT 2x20, Connector_IDC:IDC-Header_2x20_P2.54mm_Vertical, symbol cube:BUS_OUT_2x20_40__84700
- removed J20: STRAND10, Connector_JST:JST_XH_B4B-XH-A_1x04_P2.50mm_Vertical, symbol cube:STRAND10_4__75938
- removed J21: STRAND11, Connector_JST:JST_XH_B4B-XH-A_1x04_P2.50mm_Vertical, symbol cube:STRAND11_4__75938
- removed J22: STRAND12, Connector_JST:JST_XH_B4B-XH-A_1x04_P2.50mm_Vertical, symbol cube:STRAND12_4__75938
- removed J23: STRAND13, Connector_JST:JST_XH_B4B-XH-A_1x04_P2.50mm_Vertical, symbol cube:STRAND13_4__75938
- removed J24: STRAND14, Connector_JST:JST_XH_B4B-XH-A_1x04_P2.50mm_Vertical, symbol cube:STRAND14_4__75938
- removed J25: STRAND15, Connector_JST:JST_XH_B4B-XH-A_1x04_P2.50mm_Vertical, symbol cube:STRAND15_4__75938
- removed J30, J31: 12V_BUS, TerminalBlock_Phoenix:TerminalBlock_Phoenix_MKDS-1,5-2-5.08_1x02_P5.08mm_Horizontal, symbol cube:12V_BUS_2__37452
- removed JP0: ID0_SET, Jumper:SolderJumper-2_P1.3mm_Open_RoundedPad1.0x1.5mm, symbol cube:ID0_SET_2__21234
- removed JP1: ID1_SET, Jumper:SolderJumper-2_P1.3mm_Open_RoundedPad1.0x1.5mm, symbol cube:ID1_SET_2__21234
- removed JP2: ID2_SET, Jumper:SolderJumper-2_P1.3mm_Open_RoundedPad1.0x1.5mm, symbol cube:ID2_SET_2__21234
- removed JP3: ID3_SET, Jumper:SolderJumper-2_P1.3mm_Open_RoundedPad1.0x1.5mm, symbol cube:ID3_SET_2__21234
- removed JP4: ID4_SET, Jumper:SolderJumper-2_P1.3mm_Open_RoundedPad1.0x1.5mm, symbol cube:ID4_SET_2__21234
- removed JP5: ID5_SET, Jumper:SolderJumper-2_P1.3mm_Open_RoundedPad1.0x1.5mm, symbol cube:ID5_SET_2__21234
- removed L30: 1.5uH 20A, Inductor_SMD:L_TaiTech_TMPC1265_13.5x12.5mm, symbol cube:1.5uH_20A_2__21234
- removed R30, R40: 100k, Resistor_SMD:R_0603_1608Metric, symbol cube:100k_2__21234
- removed R31: 15k, Resistor_SMD:R_0603_1608Metric, symbol cube:15k_2__21234
- removed R32: 8.2k, Resistor_SMD:R_0603_1608Metric, symbol cube:8.2k_2__21234
- removed R33: 750R, Resistor_SMD:R_0603_1608Metric, symbol cube:750R_2__21234
- removed R34, R36, R39, RID0, RID1, RID2, RID3, RID4, RID5: 10k, Resistor_SMD:R_0603_1608Metric, symbol cube:10k_2__21234
- removed R35: 75k, Resistor_SMD:R_0603_1608Metric, symbol cube:75k_2__21234
- removed R37: 120k, Resistor_SMD:R_0603_1608Metric, symbol cube:120k_2__21234
- removed R38: 20k, Resistor_SMD:R_0603_1608Metric, symbol cube:20k_2__21234
- removed RC0, RC1, RC10, RC11, RC12, RC13, RC14, RC15, RC2, RC3, RC4, RC5, RC6, RC7, RC8, RC9, RD0, RD1, RD10, RD11, RD12, RD13, RD14, RD15, RD2, RD3, RD4, RD5, RD6, RD7, RD8, RD9: 33R, Resistor_SMD:R_0603_1608Metric, symbol cube:33R_2__21234
- removed U1, U2, U3, U6, U7, U8, U9: 74AHCT245PW, Package_SO:TSSOP-20_4.4x6.5mm_P0.65mm, symbol cube:74AHCT245PW_20__32821
- removed U30: TPS259474LRPWR, cube:TI_RPW0010A_VQFN-HR-10_2x2mm_P0.45mm, symbol cube:TPS259474LRPWR_10__27248
- removed U31: TPS56C215RNNR, Package_DFN_QFN:Texas_RNN0018A, symbol cube:TPS56C215RNNR_18__22882
- removed U4: 74HC688D, Package_SO:SOIC-20W_7.5x12.8mm_P1.27mm, symbol cube:74HC688D_20__12603
- removed U5: SN74AHC1G32DBVR, Package_TO_SOT_SMD:SOT-23-5, symbol cube:SN74AHC1G32DBVR_5__15265
- removed UE0, UE1, UE10, UE11, UE12, UE13, UE14, UE15, UE2, UE3, UE4, UE5, UE6, UE7, UE8, UE9: USBLC6-2SC6, Package_TO_SOT_SMD:SOT-23-6, symbol cube:USBLC6-2SC6_6__29574
- added C1, C2, C3, C36, C4, C5, C6, C7, C8, C9: 100nF, Capacitor_SMD:C_0603_1608Metric, symbol cube:100nF_2__59945
- added C10, C11, C12, C13, C14, C15: 47uF, Capacitor_SMD:C_0805_2012Metric, symbol cube:47uF_2__59945
- added C30, C31: 10nF, Capacitor_SMD:C_0603_1608Metric, symbol cube:10nF_2__59945
- added C32, C33, C34, C35: 10uF/50V, Capacitor_SMD:C_1206_3216Metric, symbol cube:10uF/50V_2__59945
- added C37: 4.7uF, Capacitor_SMD:C_0603_1608Metric, symbol cube:4.7uF_2__59945
- added C38: 22nF, Capacitor_SMD:C_0603_1608Metric, symbol cube:22nF_2__59945
- added C40, C41, C42, C43, C44, C45: 47uF/16V, Capacitor_SMD:C_1210_3225Metric, symbol cube:47uF/16V_2__59945
- added D30: SMBJ15A, Diode_SMD:D_SMB, symbol cube:SMBJ15A_2__39835
- added F10, F11, F12, F13, F14, F15, F16, F17, F18, F19, F20, F21, F22, F23, F24, F25: PTC 2A, Fuse:Fuse_1812_4532Metric, symbol cube:PTC_2A_2__59945
- added J1: BUS_IN 2x20, Connector_IDC:IDC-Header_2x20_P2.54mm_Vertical, symbol cube:BUS_IN_2x20_40__61618
- added J10: STRAND0, Connector_JST:JST_XH_B4B-XH-A_1x04_P2.50mm_Vertical, symbol cube:STRAND0_4__88812
- added J11: STRAND1, Connector_JST:JST_XH_B4B-XH-A_1x04_P2.50mm_Vertical, symbol cube:STRAND1_4__88812
- added J12: STRAND2, Connector_JST:JST_XH_B4B-XH-A_1x04_P2.50mm_Vertical, symbol cube:STRAND2_4__88812
- added J13: STRAND3, Connector_JST:JST_XH_B4B-XH-A_1x04_P2.50mm_Vertical, symbol cube:STRAND3_4__88812
- added J14: STRAND4, Connector_JST:JST_XH_B4B-XH-A_1x04_P2.50mm_Vertical, symbol cube:STRAND4_4__88812
- added J15: STRAND5, Connector_JST:JST_XH_B4B-XH-A_1x04_P2.50mm_Vertical, symbol cube:STRAND5_4__88812
- added J16: STRAND6, Connector_JST:JST_XH_B4B-XH-A_1x04_P2.50mm_Vertical, symbol cube:STRAND6_4__88812
- added J17: STRAND7, Connector_JST:JST_XH_B4B-XH-A_1x04_P2.50mm_Vertical, symbol cube:STRAND7_4__88812
- added J18: STRAND8, Connector_JST:JST_XH_B4B-XH-A_1x04_P2.50mm_Vertical, symbol cube:STRAND8_4__88812
- added J19: STRAND9, Connector_JST:JST_XH_B4B-XH-A_1x04_P2.50mm_Vertical, symbol cube:STRAND9_4__88812
- added J2: BUS_OUT 2x20, Connector_IDC:IDC-Header_2x20_P2.54mm_Vertical, symbol cube:BUS_OUT_2x20_40__61618
- added J20: STRAND10, Connector_JST:JST_XH_B4B-XH-A_1x04_P2.50mm_Vertical, symbol cube:STRAND10_4__88812
- added J21: STRAND11, Connector_JST:JST_XH_B4B-XH-A_1x04_P2.50mm_Vertical, symbol cube:STRAND11_4__88812
- added J22: STRAND12, Connector_JST:JST_XH_B4B-XH-A_1x04_P2.50mm_Vertical, symbol cube:STRAND12_4__88812
- added J23: STRAND13, Connector_JST:JST_XH_B4B-XH-A_1x04_P2.50mm_Vertical, symbol cube:STRAND13_4__88812
- added J24: STRAND14, Connector_JST:JST_XH_B4B-XH-A_1x04_P2.50mm_Vertical, symbol cube:STRAND14_4__88812
- added J25: STRAND15, Connector_JST:JST_XH_B4B-XH-A_1x04_P2.50mm_Vertical, symbol cube:STRAND15_4__88812
- added J30: 12V_BUS, TerminalBlock_Phoenix:TerminalBlock_Phoenix_MKDS-1,5-2-5.08_1x02_P5.08mm_Horizontal, symbol cube:12V_BUS_2__60152
- added JP0: ID0_SET, Jumper:SolderJumper-2_P1.3mm_Open_RoundedPad1.0x1.5mm, symbol cube:ID0_SET_2__59945
- added JP1: ID1_SET, Jumper:SolderJumper-2_P1.3mm_Open_RoundedPad1.0x1.5mm, symbol cube:ID1_SET_2__59945
- added JP2: ID2_SET, Jumper:SolderJumper-2_P1.3mm_Open_RoundedPad1.0x1.5mm, symbol cube:ID2_SET_2__59945
- added JP3: ID3_SET, Jumper:SolderJumper-2_P1.3mm_Open_RoundedPad1.0x1.5mm, symbol cube:ID3_SET_2__59945
- added JP4: ID4_SET, Jumper:SolderJumper-2_P1.3mm_Open_RoundedPad1.0x1.5mm, symbol cube:ID4_SET_2__59945
- added JP5: ID5_SET, Jumper:SolderJumper-2_P1.3mm_Open_RoundedPad1.0x1.5mm, symbol cube:ID5_SET_2__59945
- added L30: 1.5uH 20A, cube:L_YJYCOIN_YSPI1365, symbol cube:1.5uH_20A_2__59945
- added R30, R40: 100k, Resistor_SMD:R_0603_1608Metric, symbol cube:100k_2__59945
- added R31: 15k, Resistor_SMD:R_0603_1608Metric, symbol cube:15k_2__59945
- added R32: 8.2k, Resistor_SMD:R_0603_1608Metric, symbol cube:8.2k_2__59945
- added R33: 750R, Resistor_SMD:R_0603_1608Metric, symbol cube:750R_2__59945
- added R34, R36, R39, RID0, RID1, RID2, RID3, RID4, RID5: 10k, Resistor_SMD:R_0603_1608Metric, symbol cube:10k_2__59945
- added R35: 75k, Resistor_SMD:R_0603_1608Metric, symbol cube:75k_2__59945
- added R37: 120k, Resistor_SMD:R_0603_1608Metric, symbol cube:120k_2__59945
- added R38: 20k, Resistor_SMD:R_0603_1608Metric, symbol cube:20k_2__59945
- added RC0, RC1, RC10, RC11, RC12, RC13, RC14, RC15, RC2, RC3, RC4, RC5, RC6, RC7, RC8, RC9, RD0, RD1, RD10, RD11, RD12, RD13, RD14, RD15, RD2, RD3, RD4, RD5, RD6, RD7, RD8, RD9: 33R, Resistor_SMD:R_0603_1608Metric, symbol cube:33R_2__59945
- added U1, U2, U3, U6, U7, U8, U9: 74AHCT245PW, Package_SO:TSSOP-20_4.4x6.5mm_P0.65mm, symbol cube:74AHCT245PW_20__9341
- added U30: TPS259474LRPWR, cube:TI_RPW0010A_VQFN-HR-10_2x2mm_P0.45mm, symbol cube:TPS259474LRPWR_10__71391
- added U31: TPS56C215RNNR, Package_DFN_QFN:Texas_RNN0018A, symbol cube:TPS56C215RNNR_18__20520
- added U4: 74HC688D, Package_SO:SOIC-20W_7.5x12.8mm_P1.27mm, symbol cube:74HC688D_20__5331
- added U5: SN74AHC1G32DBVR, Package_TO_SOT_SMD:SOT-23-5, symbol cube:SN74AHC1G32DBVR_5__10019
- added UE0, UE1, UE10, UE11, UE12, UE13, UE14, UE15, UE2, UE3, UE4, UE5, UE6, UE7, UE8, UE9: USBLC6-2SC6, Package_TO_SOT_SMD:SOT-23-6, symbol cube:USBLC6-2SC6_6__23068
Connections:
- net +12V: now also C33.1, C34.1, C35.1, U30.6 (OUT), U31.11 (VIN_2), U31.15 (EN), U31.2 (VIN)
- net +5V: now also C1.1, C10.1, C11.1, C12.1, C13.1, C14.1, C15.1, C2.1, C3.1, C4.1, C40.1, C41.1, C42.1, C43.1, C44.1, C45.1, C5.1, C6.1, C7.1, C8.1, C9.1, F10.1, F11.1, F12.1, F13.1, F14.1, F15.1, F16.1, F17.1, F18.1, F19.1, F20.1, F21.1, F22.1, F23.1, F24.1, F25.1, L30.2, R34.2, R35.1, R39.2, RID0.1, RID1.1, RID2.1, RID3.1, RID4.1, RID5.1, U1.1 (DIR), U1.20 (VCC), U2.1 (DIR), U2.20 (VCC), U3.1 (DIR), U3.20 (VCC), U4.20 (VCC), U5.5 (VCC), U6.1 (DIR), U6.20 (VCC), U7.1 (DIR), U7.20 (VCC), U8.1 (DIR), U8.20 (VCC), U9.1 (DIR), U9.20 (VCC), UE0.5 (VBUS), UE1.5 (VBUS), UE10.5 (VBUS), UE11.5 (VBUS), UE12.5 (VBUS), UE13.5 (VBUS), UE14.5 (VBUS), UE15.5 (VBUS), UE2.5 (VBUS), UE3.5 (VBUS), UE4.5 (VBUS), UE5.5 (VBUS), UE6.5 (VBUS), UE7.5 (VBUS), UE8.5 (VBUS), UE9.5 (VBUS)
- net BST: now also C36.1, U31.1 (BOOT)
- net DVDT: now also C30.1, U30.7 (DVDT)
- net EFEN: now also R30.2, R31.1, U30.1 (EN/UVLO), U30.4 (PGTH)
- net EFOV: now also R32.1, R40.2, U30.2 (OVLO)
- net FB5: now also R35.2, R36.1, U31.13 (FB)
- net GCLK: now also U5.4 (Y), U8.2 (A1), U8.3 (A2), U8.4 (A3), U8.5 (A4), U8.6 (A5), U8.7 (A6), U8.8 (A7), U8.9 (A8), U9.2 (A1), U9.3 (A2), U9.4 (A3), U9.5 (A4), U9.6 (A5), U9.7 (A6), U9.8 (A7), U9.9 (A8)
- net GND: now also C1.2, C10.2, C11.2, C12.2, C13.2, C14.2, C15.2, C2.2, C3.2, C30.2, C31.2, C32.2, C33.2, C34.2, C35.2, C37.2, C38.2, C4.2, C40.2, C41.2, C42.2, C43.2, C44.2, C45.2, C5.2, C6.2, C7.2, C8.2, C9.2, D30.2 (A), J1.10 (GND), J1.12 (GND), J1.14 (GND), J1.16 (GND), J1.18 (GND), J1.2 (GND), J1.20 (GND), J1.22 (GND), J1.24 (GND), J1.26 (GND), J1.28 (GND), J1.30 (GND), J1.32 (GND), J1.4 (GND), J1.40 (GND), J1.6 (GND), J1.8 (GND), J10.4 (GND), J11.4 (GND), J12.4 (GND), J13.4 (GND), J14.4 (GND), J15.4 (GND), J16.4 (GND), J17.4 (GND), J18.4 (GND), J19.4 (GND), J2.10 (GND), J2.12 (GND), J2.14 (GND), J2.16 (GND), J2.18 (GND), J2.2 (GND), J2.20 (GND), J2.22 (GND), J2.24 (GND), J2.26 (GND), J2.28 (GND), J2.30 (GND), J2.32 (GND), J2.4 (GND), J2.40 (GND), J2.6 (GND), J2.8 (GND), J20.4 (GND), J21.4 (GND), J22.4 (GND), J23.4 (GND), J24.4 (GND), J25.4 (GND), J30.2 (GND), JP0.2, JP1.2, JP2.2, JP3.2, JP4.2, JP5.2, R31.2, R32.2, R33.2, R36.2, R38.2, U1.10 (GND), U1.19 (~OE), U2.10 (GND), U2.19 (~OE), U3.10 (GND), U3.19 (~OE), U3.9 (A8), U30.8 (GND), U31.10 (PGND_6), U31.12 (AGND), U31.3 (PGND), U31.4 (PGND_2), U31.5 (PGND_3), U31.8 (PGND_4), U31.9 (PGND_5), U4.1 (~G), U4.10 (GND), U4.15 (P6), U4.16 (Q6), U4.17 (P7), U4.18 (Q7), U5.3 (GND), U6.10 (GND), U6.19 (~OE), U7.10 (GND), U7.19 (~OE), U8.10 (GND), U8.19 (~OE), U9.10 (GND), U9.19 (~OE), UE0.2 (GND), UE1.2 (GND), UE10.2 (GND), UE11.2 (GND), UE12.2 (GND), UE13.2 (GND), UE14.2 (GND), UE15.2 (GND), UE2.2 (GND), UE3.2 (GND), UE4.2 (GND), UE5.2 (GND), UE6.2 (GND), UE7.2 (GND), UE8.2 (GND), UE9.2 (GND)
- net ID0: now also JP0.1, RID0.2, U4.3 (Q0)
- net ID1: now also JP1.1, RID1.2, U4.5 (Q1)
- net ID2: now also JP2.1, RID2.2, U4.7 (Q2)
- net ID3: now also JP3.1, RID3.2, U4.9 (Q3)
- net ID4: now also JP4.1, RID4.2, U4.12 (Q4)
- net ID5: now also JP5.1, RID5.2, U4.14 (Q5)
- net ILM: now also R33.1, U30.9 (ILM)
- net IN_A0: now also J1.35 (A0), U3.3 (A2)
- net IN_A1: now also J1.37 (A1), U3.4 (A3)
- net IN_A2: now also J1.39 (A2), U3.5 (A4)
- net IN_A3: now also J1.34 (A3), U3.6 (A5)
- net IN_A4: now also J1.36 (A4), U3.7 (A6)
- net IN_A5: now also J1.38 (A5), U3.8 (A7)
- net IN_CLK: now also J1.33 (CLK), U3.2 (A1)
- net IN_D0: now also J1.1 (D0), U1.2 (A1)
- net IN_D1: now also J1.3 (D1), U1.3 (A2)
- net IN_D10: now also J1.21 (D10), U2.4 (A3)
- net IN_D11: now also J1.23 (D11), U2.5 (A4)
- net IN_D12: now also J1.25 (D12), U2.6 (A5)
- net IN_D13: now also J1.27 (D13), U2.7 (A6)
- net IN_D14: now also J1.29 (D14), U2.8 (A7)
- net IN_D15: now also J1.31 (D15), U2.9 (A8)
- net IN_D2: now also J1.5 (D2), U1.4 (A3)
- net IN_D3: now also J1.7 (D3), U1.5 (A4)
- net IN_D4: now also J1.9 (D4), U1.6 (A5)
- net IN_D5: now also J1.11 (D5), U1.7 (A6)
- net IN_D6: now also J1.13 (D6), U1.8 (A7)
- net IN_D7: now also J1.15 (D7), U1.9 (A8)
- net IN_D8: now also J1.17 (D8), U2.2 (A1)
- net IN_D9: now also J1.19 (D9), U2.3 (A2)
- net ITMR: now also C31.1, U30.10 (ITIMER)
- net L_A0: now also J2.35 (A0), U3.17 (B2), U4.2 (P0)
- net L_A1: now also J2.37 (A1), U3.16 (B3), U4.4 (P1)
- net L_A2: now also J2.39 (A2), U3.15 (B4), U4.6 (P2)
- net L_A3: now also J2.34 (A3), U3.14 (B5), U4.8 (P3)
- net L_A4: now also J2.36 (A4), U3.13 (B6), U4.11 (P4)
- net L_A5: now also J2.38 (A5), U3.12 (B7), U4.13 (P5)
- net L_CLK: now also J2.33 (CLK), U3.18 (B1), U5.1 (A)
- net L_D0: now also J2.1 (D0), U1.18 (B1), U6.9 (A8)
- net L_D1: now also J2.3 (D1), U1.17 (B2), U6.8 (A7)
- net L_D10: now also J2.21 (D10), U2.16 (B3), U7.7 (A6)
- net L_D11: now also J2.23 (D11), U2.15 (B4), U7.6 (A5)
- net L_D12: now also J2.25 (D12), U2.14 (B5), U7.5 (A4)
- net L_D13: now also J2.27 (D13), U2.13 (B6), U7.4 (A3)
- net L_D14: now also J2.29 (D14), U2.12 (B7), U7.3 (A2)
- net L_D15: now also J2.31 (D15), U2.11 (B8), U7.2 (A1)
- net L_D2: now also J2.5 (D2), U1.16 (B3), U6.7 (A6)
- net L_D3: now also J2.7 (D3), U1.15 (B4), U6.6 (A5)
- net L_D4: now also J2.9 (D4), U1.14 (B5), U6.5 (A4)
- net L_D5: now also J2.11 (D5), U1.13 (B6), U6.4 (A3)
- net L_D6: now also J2.13 (D6), U1.12 (B7), U6.3 (A2)
- net L_D7: now also J2.15 (D7), U1.11 (B8), U6.2 (A1)
- net L_D8: now also J2.17 (D8), U2.18 (B1), U7.9 (A8)
- net L_D9: now also J2.19 (D9), U2.17 (B2), U7.8 (A7)
- net MODE5: now also R37.2, R38.1, U31.18 (MODE)
- net PG12: now also R34.1, U30.3 (PG)
- net PG5: now also R39.1, U31.16 (PGOOD)
- net SC0: now also J10.3 (CLK), RC0.2, UE0.3 (IO2), UE0.4 (IO2b)
- net SC1: now also J11.3 (CLK), RC1.2, UE1.3 (IO2), UE1.4 (IO2b)
- net SC10: now also J20.3 (CLK), RC10.2, UE10.3 (IO2), UE10.4 (IO2b)
- net SC11: now also J21.3 (CLK), RC11.2, UE11.3 (IO2), UE11.4 (IO2b)
- net SC12: now also J22.3 (CLK), RC12.2, UE12.3 (IO2), UE12.4 (IO2b)
- net SC13: now also J23.3 (CLK), RC13.2, UE13.3 (IO2), UE13.4 (IO2b)
- net SC14: now also J24.3 (CLK), RC14.2, UE14.3 (IO2), UE14.4 (IO2b)
- net SC15: now also J25.3 (CLK), RC15.2, UE15.3 (IO2), UE15.4 (IO2b)
- net SC2: now also J12.3 (CLK), RC2.2, UE2.3 (IO2), UE2.4 (IO2b)
- net SC3: now also J13.3 (CLK), RC3.2, UE3.3 (IO2), UE3.4 (IO2b)
- net SC4: now also J14.3 (CLK), RC4.2, UE4.3 (IO2), UE4.4 (IO2b)
- net SC5: now also J15.3 (CLK), RC5.2, UE5.3 (IO2), UE5.4 (IO2b)
- net SC6: now also J16.3 (CLK), RC6.2, UE6.3 (IO2), UE6.4 (IO2b)
- net SC7: now also J17.3 (CLK), RC7.2, UE7.3 (IO2), UE7.4 (IO2b)
- net SC8: now also J18.3 (CLK), RC8.2, UE8.3 (IO2), UE8.4 (IO2b)
- net SC9: now also J19.3 (CLK), RC9.2, UE9.3 (IO2), UE9.4 (IO2b)
- net SCR0: now also RC0.1, U8.11 (B8)
- net SCR1: now also RC1.1, U8.12 (B7)
- net SCR10: now also RC10.1, U9.13 (B6)
- net SCR11: now also RC11.1, U9.14 (B5)
- net SCR12: now also RC12.1, U9.15 (B4)
- net SCR13: now also RC13.1, U9.16 (B3)
- net SCR14: now also RC14.1, U9.17 (B2)
- net SCR15: now also RC15.1, U9.18 (B1)
- net SCR2: now also RC2.1, U8.13 (B6)
- net SCR3: now also RC3.1, U8.14 (B5)
- net SCR4: now also RC4.1, U8.15 (B4)
- net SCR5: now also RC5.1, U8.16 (B3)
- net SCR6: now also RC6.1, U8.17 (B2)
- net SCR7: now also RC7.1, U8.18 (B1)
- net SCR8: now also RC8.1, U9.11 (B8)
- net SCR9: now also RC9.1, U9.12 (B7)
- net SD0: now also J10.2 (DATA), RD0.2, UE0.1 (IO1), UE0.6 (IO1b)
- net SD1: now also J11.2 (DATA), RD1.2, UE1.1 (IO1), UE1.6 (IO1b)
- net SD10: now also J20.2 (DATA), RD10.2, UE10.1 (IO1), UE10.6 (IO1b)
- net SD11: now also J21.2 (DATA), RD11.2, UE11.1 (IO1), UE11.6 (IO1b)
- net SD12: now also J22.2 (DATA), RD12.2, UE12.1 (IO1), UE12.6 (IO1b)
- net SD13: now also J23.2 (DATA), RD13.2, UE13.1 (IO1), UE13.6 (IO1b)
- net SD14: now also J24.2 (DATA), RD14.2, UE14.1 (IO1), UE14.6 (IO1b)
- net SD15: now also J25.2 (DATA), RD15.2, UE15.1 (IO1), UE15.6 (IO1b)
- net SD2: now also J12.2 (DATA), RD2.2, UE2.1 (IO1), UE2.6 (IO1b)
- net SD3: now also J13.2 (DATA), RD3.2, UE3.1 (IO1), UE3.6 (IO1b)
- net SD4: now also J14.2 (DATA), RD4.2, UE4.1 (IO1), UE4.6 (IO1b)
- net SD5: now also J15.2 (DATA), RD5.2, UE5.1 (IO1), UE5.6 (IO1b)
- net SD6: now also J16.2 (DATA), RD6.2, UE6.1 (IO1), UE6.6 (IO1b)
- net SD7: now also J17.2 (DATA), RD7.2, UE7.1 (IO1), UE7.6 (IO1b)
- net SD8: now also J18.2 (DATA), RD8.2, UE8.1 (IO1), UE8.6 (IO1b)
- net SD9: now also J19.2 (DATA), RD9.2, UE9.1 (IO1), UE9.6 (IO1b)
- net SDR0: now also RD0.1, U6.11 (B8)
- net SDR1: now also RD1.1, U6.12 (B7)
- net SDR10: now also RD10.1, U7.13 (B6)
- net SDR11: now also RD11.1, U7.14 (B5)
- net SDR12: now also RD12.1, U7.15 (B4)
- net SDR13: now also RD13.1, U7.16 (B3)
- net SDR14: now also RD14.1, U7.17 (B2)
- net SDR15: now also RD15.1, U7.18 (B1)
- net SDR2: now also RD2.1, U6.13 (B6)
- net SDR3: now also RD3.1, U6.14 (B5)
- net SDR4: now also RD4.1, U6.15 (B4)
- net SDR5: now also RD5.1, U6.16 (B3)
- net SDR6: now also RD6.1, U6.17 (B2)
- net SDR7: now also RD7.1, U6.18 (B1)
- net SDR8: now also RD8.1, U7.11 (B8)
- net SDR9: now also RD9.1, U7.12 (B7)
- net SEL_N: now also U4.19 (~P=Q), U5.2 (B)
- net SS5: now also C38.1, U31.14 (SS)
- net SW5: now also C36.2, L30.1, U31.6 (SW), U31.7 (SW_2)
- net V12_IN: now also C32.1, D30.1 (K), J30.1 (+12V), R30.1, R40.1, U30.5 (IN)
- net V5S0: now also F10.2, J10.1 (+5V)
- net V5S1: now also F11.2, J11.1 (+5V)
- net V5S10: now also F20.2, J20.1 (+5V)
- net V5S11: now also F21.2, J21.1 (+5V)
- net V5S12: now also F22.2, J22.1 (+5V)
- net V5S13: now also F23.2, J23.1 (+5V)
- net V5S14: now also F24.2, J24.1 (+5V)
- net V5S15: now also F25.2, J25.1 (+5V)
- net V5S2: now also F12.2, J12.1 (+5V)
- net V5S3: now also F13.2, J13.1 (+5V)
- net V5S4: now also F14.2, J14.1 (+5V)
- net V5S5: now also F15.2, J15.1 (+5V)
- net V5S6: now also F16.2, J16.1 (+5V)
- net V5S7: now also F17.2, J17.1 (+5V)
- net V5S8: now also F18.2, J18.1 (+5V)
- net V5S9: now also F19.2, J19.1 (+5V)
- net VREG5: now also C37.1, R37.1, U31.17 (VREG5)
