File: hardware/branch_v1/branch_v1.kicad_pcb (KiCad board)
At the start: 2 copper layers, 250 x 100 mm, 156 parts, among them J1 BUS_IN 2x20, J10 STRAND0, J11 STRAND1, J12 STRAND2, J13 STRAND3, J14 STRAND4, J15 STRAND5, J16 STRAND6, J17 STRAND7, J18 STRAND8, J19 STRAND9, J2 BUS_OUT 2x20, J20 STRAND10, J21 STRAND11, J22 STRAND12, J23 STRAND13, J24 STRAND14, J25 STRAND15, J30 12V_BUS, U1 74AHCT245PW, U2 74AHCT245PW, U3 74AHCT245PW, U30 TPS259474LRPWR, U31 TPS56C215RNNR, U4 74HC688D, U5 SN74AHC1G32DBVR, U6 74AHCT245PW, U7 74AHCT245PW, U8 74AHCT245PW, U9 74AHCT245PW

Commit message: 1 m strip board: JLC limit check, 4x250 mm segments, parametric schematic (124/64/48/32, ERC 0), strip power/current calc; main fab+3D renders; fetch3d, fab.sh; docs
Parts:
- moved H2 76.0 mm to (246.0, 80.0)
- moved H1 36.0 mm to (4.00, 40.0)
- moved F25 7.50 mm to (213.0, 82.5)
- moved J25 7.50 mm to (214.5, 93.0)
- moved RC15 7.50 mm to (219.5, 78.0)
- moved RD15 7.50 mm to (217.0, 78.0)
- moved UE15 7.50 mm to (218.2, 85.0)
- moved C15 7.00 mm to (210.2, 71.5)
- moved F24 7.00 mm to (199.5, 82.5)
- moved J24 7.00 mm to (201.0, 93.0)
- moved RC14 7.00 mm to (206.0, 78.0)
- moved RD14 7.00 mm to (203.5, 78.0)
- moved UE14 7.00 mm to (204.8, 85.0)
- moved F23 6.50 mm to (186.0, 82.5)
- moved J23 6.50 mm to (187.5, 93.0)
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Routing:
- net /GND: track 115.5 -> 61.1 mm, vias 299 -> 78
- net /ID5: track 11.6 -> 65.4 mm, vias 0 -> 2
- net /ID1: track 11.6 -> 58.1 mm, vias 0 -> 2
- net /L_A1: track 91.0 -> 59.0 mm, vias 3 -> 2
- net /L_A0: track 86.3 -> 59.1 mm, vias 3 -> 2
- net /ID2: track 59.9 -> 83.1 mm
- net /IN_D4: track 35.8 -> 23.3 mm, vias 0 -> 1
- net /+5V: track 128.9 -> 116.8 mm, vias 62 -> 93
- net /L_A5: track 101.8 -> 110.0 mm
- net /IN_D3: track 26.0 -> 33.6 mm, vias 1 -> 0
- net /SDR15: track 71.9 -> 79.4 mm
- net /SCR15: track 88.4 -> 95.9 mm
- net /ID3: track 66.8 -> 74.0 mm
- net /SCR14: track 76.1 -> 83.1 mm
- net /SDR14: track 59.6 -> 66.6 mm
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