File: hardware/main_v1/main_v1.kicad_sch (KiCad schematic)
At the start: 82 parts, among them J1 PORT0, J10 12V_IN, J2 PORT1, J3 PORT2, J4 PORT3, J5 PORT4, J6 PORT5, J7 PORT6, J8 PORT7, J9 USB-C, SW1 BOOT, SW2 RESET, U1 ESP32-S3-WROOM-1-N16R8, U10 74LVC245APW, U11 74LVC245APW, U12 74LVC245APW, U13 74LVC245APW, U14 74LVC245APW, U15 74LVC245APW, U16 74LVC245APW, U17 74LVC245APW, U18 74LVC245APW, U19 74LVC245APW, U2 AP63203WU-7, U20 74LVC245APW, U21 74LVC245APW, U22 74LVC245APW, U23 74LVC245APW, U24 74LVC245APW, U25 74LVC245APW, U26 74LVC245APW, U27 74LVC245APW, U28 74LVC245APW, U29 74LVC245APW, U3 USBLC6-2SC6, U30 74LVC245APW, U31 74LVC245APW, U32 74LVC245APW, U33 74LVC245APW

Commit message: Size table + pixel choice, cube footprint lib (TPS25947 RPW, verified inductors), schematic->PCB linking (main parity 0), TPD4E05U06 port ESD, branch layout WIP
Parts:
- removed C1: 10uF50V, Capacitor_SMD:C_1206_3216Metric, symbol cube:10uF50V_2__64643
- removed C10, C11, C12, C13, C14, C15, C16, C17, C18, C19, C2, C20, C21, C22, C23, C24, C25, C26, C27, C28, C29, C30, C31, C32, C33, C5, C7: 100nF, Capacitor_SMD:C_0603_1608Metric, symbol cube:100nF_2__64643
- removed C3, C4: 22uF, Capacitor_SMD:C_0603_1608Metric, symbol cube:22uF_2__64643
- removed C6: 1uF, Capacitor_SMD:C_0603_1608Metric, symbol cube:1uF_2__64643
- removed C8: 47uF, Capacitor_SMD:C_1210_3225Metric, symbol cube:47uF_2__64643
- removed D1: SS34, Diode_SMD:D_SMA, symbol cube:SS34_2__64643
- removed D2: STATUS, LED_SMD:LED_0603_1608Metric, symbol cube:STATUS_2__64643
- removed D3: SS34 (rev.pol.), Diode_SMD:D_SMA, symbol cube:SS34_(rev.pol.)_2__64643
- removed D4: SMBJ15A, Diode_SMD:D_SMB, symbol cube:SMBJ15A_2__64643
- removed F1: PTC 2A/16V, Fuse:Fuse_1812_4532Metric, symbol cube:PTC_2A/16V_2__64643
- removed J1: PORT0, Connector_IDC:IDC-Header_2x20_P2.54mm_Vertical, symbol cube:PORT0_40__64544
- removed J10: 12V_IN, TerminalBlock_Phoenix:TerminalBlock_Phoenix_MKDS-1,5-2-5.08_1x02_P5.08mm_Horizontal, symbol cube:12V_IN_2__64643
- removed J2: PORT1, Connector_IDC:IDC-Header_2x20_P2.54mm_Vertical, symbol cube:PORT1_40__64544
- removed J3: PORT2, Connector_IDC:IDC-Header_2x20_P2.54mm_Vertical, symbol cube:PORT2_40__64544
- removed J4: PORT3, Connector_IDC:IDC-Header_2x20_P2.54mm_Vertical, symbol cube:PORT3_40__64544
- removed J5: PORT4, Connector_IDC:IDC-Header_2x20_P2.54mm_Vertical, symbol cube:PORT4_40__64544
- removed J6: PORT5, Connector_IDC:IDC-Header_2x20_P2.54mm_Vertical, symbol cube:PORT5_40__64544
- removed J7: PORT6, Connector_IDC:IDC-Header_2x20_P2.54mm_Vertical, symbol cube:PORT6_40__64544
- removed J8: PORT7, Connector_IDC:IDC-Header_2x20_P2.54mm_Vertical, symbol cube:PORT7_40__64544
- removed J9: USB-C, Connector_USB:USB_C_Receptacle_HRO_TYPE-C-31-M-12, symbol cube:USB-C_17__71995
- removed L1: 3.3uH, Inductor_SMD:L_Bourns_SRP7028A_7.3x6.6mm, symbol cube:3.3uH_2__64643
- removed R1, R4: 10k, Resistor_SMD:R_0603_1608Metric, symbol cube:10k_2__64643
- removed R2, R3: 5.1k, Resistor_SMD:R_0603_1608Metric, symbol cube:5.1k_2__64643
- removed R5: 1k, Resistor_SMD:R_0603_1608Metric, symbol cube:1k_2__64643
- removed SW1: BOOT, Button_Switch_SMD:SW_Push_1P1T_XKB_TS-1187A, symbol cube:BOOT_2__64643
- removed SW2: RESET, Button_Switch_SMD:SW_Push_1P1T_XKB_TS-1187A, symbol cube:RESET_2__64643
- removed U1: ESP32-S3-WROOM-1-N16R8, RF_Module:ESP32-S3-WROOM-1, symbol cube:ESP32-S3-WROOM-1-N16R8_41__28950
- removed U10, U11, U12, U13, U14, U15, U16, U17, U18, U19, U20, U21, U22, U23, U24, U25, U26, U27, U28, U29, U30, U31, U32, U33: 74LVC245APW, Package_SO:TSSOP-20_4.4x6.5mm_P0.65mm, symbol cube:74LVC245APW_20__14351
- removed U2: AP63203WU-7, Package_TO_SOT_SMD:TSOT-23-6, symbol cube:AP63203WU-7_6__41926
- removed U3: USBLC6-2SC6, Package_TO_SOT_SMD:SOT-23-6, symbol cube:USBLC6-2SC6_6__41926
- added C1: 10uF50V, Capacitor_SMD:C_1206_3216Metric, symbol cube:10uF50V_2__83787
- added C10, C11, C12, C13, C14, C15, C16, C17, C18, C19, C2, C20, C21, C22, C23, C24, C25, C26, C27, C28, C29, C30, C31, C32, C33, C5, C7: 100nF, Capacitor_SMD:C_0603_1608Metric, symbol cube:100nF_2__83787
- added C3, C4: 22uF, Capacitor_SMD:C_0603_1608Metric, symbol cube:22uF_2__83787
- added C6: 1uF, Capacitor_SMD:C_0603_1608Metric, symbol cube:1uF_2__83787
- added C8: 47uF, Capacitor_SMD:C_1210_3225Metric, symbol cube:47uF_2__83787
- added D1: SS34, Diode_SMD:D_SMA, symbol cube:SS34_2__83787
- added D2: STATUS, LED_SMD:LED_0603_1608Metric, symbol cube:STATUS_2__83787
- added D3: SS34 (rev.pol.), Diode_SMD:D_SMA, symbol cube:SS34_(rev.pol.)_2__83787
- added D4: SMBJ15A, Diode_SMD:D_SMB, symbol cube:SMBJ15A_2__83787
- added F1: PTC 2A/16V, Fuse:Fuse_1812_4532Metric, symbol cube:PTC_2A/16V_2__83787
- added J1: PORT0, Connector_IDC:IDC-Header_2x20_P2.54mm_Vertical, symbol cube:PORT0_40__9015
- added J10: 12V_IN, TerminalBlock_Phoenix:TerminalBlock_Phoenix_MKDS-1,5-2-5.08_1x02_P5.08mm_Horizontal, symbol cube:12V_IN_2__83787
- added J2: PORT1, Connector_IDC:IDC-Header_2x20_P2.54mm_Vertical, symbol cube:PORT1_40__9015
- added J3: PORT2, Connector_IDC:IDC-Header_2x20_P2.54mm_Vertical, symbol cube:PORT2_40__9015
- added J4: PORT3, Connector_IDC:IDC-Header_2x20_P2.54mm_Vertical, symbol cube:PORT3_40__9015
- added J5: PORT4, Connector_IDC:IDC-Header_2x20_P2.54mm_Vertical, symbol cube:PORT4_40__9015
- added J6: PORT5, Connector_IDC:IDC-Header_2x20_P2.54mm_Vertical, symbol cube:PORT5_40__9015
- added J7: PORT6, Connector_IDC:IDC-Header_2x20_P2.54mm_Vertical, symbol cube:PORT6_40__9015
- added J8: PORT7, Connector_IDC:IDC-Header_2x20_P2.54mm_Vertical, symbol cube:PORT7_40__9015
- added J9: USB-C, Connector_USB:USB_C_Receptacle_HRO_TYPE-C-31-M-12, symbol cube:USB-C_17__25943
- added L1: 3.3uH, cube:L_Cjiang_FXL0630, symbol cube:3.3uH_2__83787
- added R1, R4: 10k, Resistor_SMD:R_0603_1608Metric, symbol cube:10k_2__83787
- added R2, R3: 5.1k, Resistor_SMD:R_0603_1608Metric, symbol cube:5.1k_2__83787
- added R5: 1k, Resistor_SMD:R_0603_1608Metric, symbol cube:1k_2__83787
- added SW1: BOOT, Button_Switch_SMD:SW_Push_1P1T_XKB_TS-1187A, symbol cube:BOOT_2__83787
- added SW2: RESET, Button_Switch_SMD:SW_Push_1P1T_XKB_TS-1187A, symbol cube:RESET_2__83787
- added U1: ESP32-S3-WROOM-1-N16R8, RF_Module:ESP32-S3-WROOM-1, symbol cube:ESP32-S3-WROOM-1-N16R8_41__2323
- added U10, U11, U12, U13, U14, U15, U16, U17, U18, U19, U20, U21, U22, U23, U24, U25, U26, U27, U28, U29, U30, U31, U32, U33: 74LVC245APW, Package_SO:TSSOP-20_4.4x6.5mm_P0.65mm, symbol cube:74LVC245APW_20__5531
- added U2: AP63203WU-7, Package_TO_SOT_SMD:TSOT-23-6, symbol cube:AP63203WU-7_6__28962
- added U3: USBLC6-2SC6, Package_TO_SOT_SMD:SOT-23-6, symbol cube:USBLC6-2SC6_6__28962
- added UE0, UE1, UE10, UE11, UE12, UE13, UE14, UE15, UE2, UE20, UE21, UE22, UE23, UE24, UE25, UE3, UE30, UE31, UE32, UE33, UE34, UE35, UE4, UE40, UE41, UE42, UE43, UE44, UE45, UE5, UE50, UE51, UE52, UE53, UE54, UE55, UE60, UE61, UE62, UE63, UE64, UE65, UE70, UE71, UE72, UE73, UE74, UE75: TPD4E05U06DQAR, Package_SON:USON-10_2.5x1.0mm_P0.5mm, symbol cube:TPD4E05U06DQAR_10__83139
Connections:
- net +3V3: now also C10.2, C11.2, C12.2, C13.2, C14.2, C15.2, C16.2, C17.2, C18.2, C19.2, C20.2, C21.2, C22.1, C23.1, C24.1, C25.1, C26.1, C27.1, C28.1, C29.1, C3.1, C30.1, C31.1, C32.1, C33.1, C4.1, C5.1, C8.1, L1.2, R1.2, R4.2, U1.2, U10.1, U10.20, U11.1, U11.20, U12.1, U12.20, U13.1, U13.20, U14.1, U14.20, U15.1, U15.20, U16.1, U16.20, U17.1, U17.20, U18.1, U18.20, U19.1, U19.20, U2.1, U20.1, U20.20, U21.1, U21.20, U22.1, U22.20, U23.1, U23.20, U24.1, U24.20, U25.1, U25.20, U26.1, U26.20, U27.1, U27.20, U28.1, U28.20, U29.1, U29.20, U30.1, U30.20, U31.1, U31.20, U32.1, U32.20, U33.1, U33.20
- net A0: now also U1.11, U12.4, U15.4, U18.4, U21.4, U24.4, U27.4, U30.4, U33.4
- net A1: now also U1.10, U12.6, U15.6, U18.6, U21.6, U24.6, U27.6, U30.6, U33.6
- net A2: now also U1.9, U12.8, U15.8, U18.8, U21.8, U24.8, U27.8, U30.8, U33.8
- net A3: now also U1.8, U12.3, U15.3, U18.3, U21.3, U24.3, U27.3, U30.3, U33.3
- net A4: now also U1.7, U12.5, U15.5, U18.5, U21.5, U24.5, U27.5, U30.5, U33.5
- net A5: now also U1.6, U12.7, U15.7, U18.7, U21.7, U24.7, U27.7, U30.7, U33.7
- net BST: now also C7.2, U2.6
- net CC1: now also J9.A5, R2.1
- net CC2: now also J9.B5, R3.1
- net CLK: now also U1.12, U12.2, U15.2, U18.2, U21.2, U24.2, U27.2, U30.2, U33.2
- net D0: now also U1.39, U10.2, U13.2, U16.2, U19.2, U22.2, U25.2, U28.2, U31.2
- net D1: now also U1.38, U10.3, U13.3, U16.3, U19.3, U22.3, U25.3, U28.3, U31.3
- net D10: now also U1.22, U11.4, U14.4, U17.4, U20.4, U23.4, U26.4, U29.4, U32.4
- net D11: now also U1.21, U11.5, U14.5, U17.5, U20.5, U23.5, U26.5, U29.5, U32.5
- net D12: now also U1.20, U11.6, U14.6, U17.6, U20.6, U23.6, U26.6, U29.6, U32.6
- net D13: now also U1.19, U11.7, U14.7, U17.7, U20.7, U23.7, U26.7, U29.7, U32.7
- net D14: now also U1.18, U11.8, U14.8, U17.8, U20.8, U23.8, U26.8, U29.8, U32.8
- net D15: now also U1.17, U11.9, U14.9, U17.9, U20.9, U23.9, U26.9, U29.9, U32.9
- net D2: now also U1.35, U10.4, U13.4, U16.4, U19.4, U22.4, U25.4, U28.4, U31.4
- net D3: now also U1.34, U10.5, U13.5, U16.5, U19.5, U22.5, U25.5, U28.5, U31.5
- net D4: now also U1.33, U10.6, U13.6, U16.6, U19.6, U22.6, U25.6, U28.6, U31.6
- net D5: now also U1.32, U10.7, U13.7, U16.7, U19.7, U22.7, U25.7, U28.7, U31.7
- net D6: now also U1.31, U10.8, U13.8, U16.8, U19.8, U22.8, U25.8, U28.8, U31.8
- net D7: now also U1.25, U10.9, U13.9, U16.9, U19.9, U22.9, U25.9, U28.9, U31.9
- net D8: now also U1.24, U11.2, U14.2, U17.2, U20.2, U23.2, U26.2, U29.2, U32.2
- net D9: now also U1.23, U11.3, U14.3, U17.3, U20.3, U23.3, U26.3, U29.3, U32.3
- net EN: now also C6.1, R1.1, SW2.1, U1.3
- net GND: now also C1.2, C10.1, C11.1, C12.1, C13.1, C14.1, C15.1, C16.1, C17.1, C18.1, C19.1, C2.2, C20.1, C21.1, C22.2, C23.2, C24.2, C25.2, C26.2, C27.2, C28.2, C29.2, C3.2, C30.2, C31.2, C32.2, C33.2, C4.2, C5.2, C6.2, C8.2, D2.1, D4.2, J1.10, J1.12, J1.14, J1.16, J1.18, J1.2, J1.20, J1.22, J1.24, J1.26, J1.28, J1.30, J1.32, J1.4, J1.40, J1.6, J1.8, J10.2, J2.10, J2.12, J2.14, J2.16, J2.18, J2.2, J2.20, J2.22, J2.24, J2.26, J2.28, J2.30, J2.32, J2.4, J2.40, J2.6, J2.8, J3.10, J3.12, J3.14, J3.16, J3.18, J3.2, J3.20, J3.22, J3.24, J3.26, J3.28, J3.30, J3.32, J3.4, J3.40, J3.6, J3.8, J4.10, J4.12, J4.14, J4.16, J4.18, J4.2, J4.20, J4.22, J4.24, J4.26, J4.28, J4.30, J4.32, J4.4, J4.40, J4.6, J4.8, J5.10, J5.12, J5.14, J5.16, J5.18, J5.2, J5.20, J5.22, J5.24, J5.26, J5.28, J5.30, J5.32, J5.4, J5.40, J5.6, J5.8, J6.10, J6.12, J6.14, J6.16, J6.18, J6.2, J6.20, J6.22, J6.24, J6.26, J6.28, J6.30, J6.32, J6.4, J6.40, J6.6, J6.8, J7.10, J7.12, J7.14, J7.16, J7.18, J7.2, J7.20, J7.22, J7.24, J7.26, J7.28, J7.30, J7.32, J7.4, J7.40, J7.6, J7.8, J8.10, J8.12, J8.14, J8.16, J8.18, J8.2, J8.20, J8.22, J8.24, J8.26, J8.28, J8.30, J8.32, J8.4, J8.40, J8.6, J8.8, J9.A1, J9.A12, J9.A8, J9.B1, J9.B12, J9.B8, J9.SH, R2.2, R3.2, SW1.2, SW2.2, U1.1, U1.40, U1.41, U10.10, U11.10, U12.10, U12.9, U13.10, U14.10, U15.10, U15.9, U16.10, U17.10, U18.10, U18.9, U19.10, U2.4, U20.10, U21.10, U21.9, U22.10, U23.10, U24.10, U24.9, U25.10, U26.10, U27.10, U27.9, U28.10, U29.10, U3.2, U30.10, U30.9, U31.10, U32.10, U33.10, U33.9, UE0.3, UE0.8, UE1.3, UE1.8, UE10.3, UE10.8, UE11.3, UE11.8, UE12.3, UE12.8, UE13.3, UE13.8, UE14.3, UE14.8, UE15.3, UE15.8, UE2.3, UE2.8, UE20.3, UE20.8, UE21.3, UE21.8, UE22.3, UE22.8, UE23.3, UE23.8, UE24.3, UE24.8, UE25.3, UE25.8, UE3.3, UE3.8, UE30.3, UE30.8, UE31.3, UE31.8, UE32.3, UE32.8, UE33.3, UE33.8, UE34.3, UE34.8, UE35.3, UE35.8, UE4.3, UE4.8, UE40.3, UE40.8, UE41.3, UE41.8, UE42.3, UE42.8, UE43.3, UE43.8, UE44.3, UE44.8, UE45.3, UE45.8, UE5.3, UE5.8, UE50.3, UE50.8, UE51.3, UE51.8, UE52.3, UE52.8, UE53.3, UE53.8, UE54.3, UE54.8, UE55.3, UE55.8, UE60.3, UE60.8, UE61.3, UE61.8, UE62.3, UE62.8, UE63.3, UE63.8, UE64.3, UE64.8, UE65.3, UE65.8, UE70.3, UE70.8, UE71.3, UE71.8, UE72.3, UE72.8, UE73.3, UE73.8, UE74.3, UE74.8, UE75.3, UE75.8
- net IO0: now also SW1.1, U1.27
- net LED: now also R5.1, U1.4
- net LED_K: now also D2.2, R5.2
- net OE_N: now also R4.1, U1.5, U10.19, U11.19, U12.19, U13.19, U14.19, U15.19, U16.19, U17.19, U18.19, U19.19, U20.19, U21.19, U22.19, U23.19, U24.19, U25.19, U26.19, U27.19, U28.19, U29.19, U30.19, U31.19, U32.19, U33.19
- net P0_A0: now also J1.35, U12.16, UE4.2
- net P0_A1: now also J1.37, U12.14, UE4.4
- net P0_A2: now also J1.39, U12.12, UE4.5
- net P0_A3: now also J1.34, U12.17, UE5.5
- net P0_A4: now also J1.36, U12.15, UE5.4
- net P0_A5: now also J1.38, U12.13, UE5.2
- net P0_CLK: now also J1.33, U12.18, UE4.1
- net P0_D0: now also J1.1, U10.18, UE0.1
- net P0_D1: now also J1.3, U10.17, UE0.2
- net P0_D10: now also J1.21, U11.16, UE2.4
- net P0_D11: now also J1.23, U11.15, UE2.5
- net P0_D12: now also J1.25, U11.14, UE3.1
- net P0_D13: now also J1.27, U11.13, UE3.2
- net P0_D14: now also J1.29, U11.12, UE3.4
- net P0_D15: now also J1.31, U11.11, UE3.5
- net P0_D2: now also J1.5, U10.16, UE0.4
- net P0_D3: now also J1.7, U10.15, UE0.5
- net P0_D4: now also J1.9, U10.14, UE1.1
- net P0_D5: now also J1.11, U10.13, UE1.2
- net P0_D6: now also J1.13, U10.12, UE1.4
- net P0_D7: now also J1.15, U10.11, UE1.5
- net P0_D8: now also J1.17, U11.18, UE2.1
- net P0_D9: now also J1.19, U11.17, UE2.2
- net P1_A0: now also J2.35, U15.16, UE14.2
- net P1_A1: now also J2.37, U15.14, UE14.4
- net P1_A2: now also J2.39, U15.12, UE14.5
- net P1_A3: now also J2.34, U15.17, UE15.5
- net P1_A4: now also J2.36, U15.15, UE15.4
- net P1_A5: now also J2.38, U15.13, UE15.2
- net P1_CLK: now also J2.33, U15.18, UE14.1
- net P1_D0: now also J2.1, U13.18, UE10.1
- net P1_D1: now also J2.3, U13.17, UE10.2
- net P1_D10: now also J2.21, U14.16, UE12.4
- net P1_D11: now also J2.23, U14.15, UE12.5
- net P1_D12: now also J2.25, U14.14, UE13.1
- net P1_D13: now also J2.27, U14.13, UE13.2
- net P1_D14: now also J2.29, U14.12, UE13.4
- net P1_D15: now also J2.31, U14.11, UE13.5
- net P1_D2: now also J2.5, U13.16, UE10.4
- net P1_D3: now also J2.7, U13.15, UE10.5
- net P1_D4: now also J2.9, U13.14, UE11.1
- net P1_D5: now also J2.11, U13.13, UE11.2
- net P1_D6: now also J2.13, U13.12, UE11.4
- net P1_D7: now also J2.15, U13.11, UE11.5
- net P1_D8: now also J2.17, U14.18, UE12.1
- net P1_D9: now also J2.19, U14.17, UE12.2
- net P2_A0: now also J3.35, U18.16, UE24.2
- net P2_A1: now also J3.37, U18.14, UE24.4
- net P2_A2: now also J3.39, U18.12, UE24.5
- net P2_A3: now also J3.34, U18.17, UE25.5
- net P2_A4: now also J3.36, U18.15, UE25.4
- net P2_A5: now also J3.38, U18.13, UE25.2
- net P2_CLK: now also J3.33, U18.18, UE24.1
- net P2_D0: now also J3.1, U16.18, UE20.1
- net P2_D1: now also J3.3, U16.17, UE20.2
- net P2_D10: now also J3.21, U17.16, UE22.4
- net P2_D11: now also J3.23, U17.15, UE22.5
- net P2_D12: now also J3.25, U17.14, UE23.1
- net P2_D13: now also J3.27, U17.13, UE23.2
- net P2_D14: now also J3.29, U17.12, UE23.4
- net P2_D15: now also J3.31, U17.11, UE23.5
- net P2_D2: now also J3.5, U16.16, UE20.4
- net P2_D3: now also J3.7, U16.15, UE20.5
- net P2_D4: now also J3.9, U16.14, UE21.1
- net P2_D5: now also J3.11, U16.13, UE21.2
- net P2_D6: now also J3.13, U16.12, UE21.4
- net P2_D7: now also J3.15, U16.11, UE21.5
- net P2_D8: now also J3.17, U17.18, UE22.1
- net P2_D9: now also J3.19, U17.17, UE22.2
- net P3_A0: now also J4.35, U21.16, UE34.2
- net P3_A1: now also J4.37, U21.14, UE34.4
- net P3_A2: now also J4.39, U21.12, UE34.5
- net P3_A3: now also J4.34, U21.17, UE35.5
- net P3_A4: now also J4.36, U21.15, UE35.4
- net P3_A5: now also J4.38, U21.13, UE35.2
- net P3_CLK: now also J4.33, U21.18, UE34.1
- net P3_D0: now also J4.1, U19.18, UE30.1
- net P3_D1: now also J4.3, U19.17, UE30.2
- net P3_D10: now also J4.21, U20.16, UE32.4
- net P3_D11: now also J4.23, U20.15, UE32.5
- net P3_D12: now also J4.25, U20.14, UE33.1
- net P3_D13: now also J4.27, U20.13, UE33.2
- net P3_D14: now also J4.29, U20.12, UE33.4
- net P3_D15: now also J4.31, U20.11, UE33.5
- net P3_D2: now also J4.5, U19.16, UE30.4
- net P3_D3: now also J4.7, U19.15, UE30.5
- net P3_D4: now also J4.9, U19.14, UE31.1
- net P3_D5: now also J4.11, U19.13, UE31.2
- net P3_D6: now also J4.13, U19.12, UE31.4
- net P3_D7: now also J4.15, U19.11, UE31.5
- net P3_D8: now also J4.17, U20.18, UE32.1
- net P3_D9: now also J4.19, U20.17, UE32.2
- net P4_A0: now also J5.35, U24.16, UE44.2
- net P4_A1: now also J5.37, U24.14, UE44.4
- net P4_A2: now also J5.39, U24.12, UE44.5
- net P4_A3: now also J5.34, U24.17, UE45.4
- net P4_A4: now also J5.36, U24.15, UE45.2
- net P4_A5: now also J5.38, U24.13, UE45.1
- net P4_CLK: now also J5.33, U24.18, UE44.1
- net P4_D0: now also J5.1, U22.18, UE40.1
- net P4_D1: now also J5.3, U22.17, UE40.2
- net P4_D10: now also J5.21, U23.16, UE42.4
- net P4_D11: now also J5.23, U23.15, UE42.5
- net P4_D12: now also J5.25, U23.14, UE43.1
- net P4_D13: now also J5.27, U23.13, UE43.2
- net P4_D14: now also J5.29, U23.12, UE43.4
- net P4_D15: now also J5.31, U23.11, UE43.5
- net P4_D2: now also J5.5, U22.16, UE40.4
- net P4_D3: now also J5.7, U22.15, UE40.5
- net P4_D4: now also J5.9, U22.14, UE41.1
- net P4_D5: now also J5.11, U22.13, UE41.2
- net P4_D6: now also J5.13, U22.12, UE41.4
- net P4_D7: now also J5.15, U22.11, UE41.5
- net P4_D8: now also J5.17, U23.18, UE42.1
- net P4_D9: now also J5.19, U23.17, UE42.2
- net P5_A0: now also J6.35, U27.16, UE54.2
- net P5_A1: now also J6.37, U27.14, UE54.4
- net P5_A2: now also J6.39, U27.12, UE54.5
- net P5_A3: now also J6.34, U27.17, UE55.4
- net P5_A4: now also J6.36, U27.15, UE55.2
- net P5_A5: now also J6.38, U27.13, UE55.1
- net P5_CLK: now also J6.33, U27.18, UE54.1
- net P5_D0: now also J6.1, U25.18, UE50.1
- net P5_D1: now also J6.3, U25.17, UE50.2
- net P5_D10: now also J6.21, U26.16, UE52.4
- net P5_D11: now also J6.23, U26.15, UE52.5
- net P5_D12: now also J6.25, U26.14, UE53.1
- net P5_D13: now also J6.27, U26.13, UE53.2
- net P5_D14: now also J6.29, U26.12, UE53.4
- net P5_D15: now also J6.31, U26.11, UE53.5
- net P5_D2: now also J6.5, U25.16, UE50.4
- net P5_D3: now also J6.7, U25.15, UE50.5
- net P5_D4: now also J6.9, U25.14, UE51.1
- net P5_D5: now also J6.11, U25.13, UE51.2
- net P5_D6: now also J6.13, U25.12, UE51.4
- net P5_D7: now also J6.15, U25.11, UE51.5
- net P5_D8: now also J6.17, U26.18, UE52.1
- net P5_D9: now also J6.19, U26.17, UE52.2
- net P6_A0: now also J7.35, U30.16, UE64.2
- net P6_A1: now also J7.37, U30.14, UE64.4
- net P6_A2: now also J7.39, U30.12, UE64.5
- net P6_A3: now also J7.34, U30.17, UE65.4
- net P6_A4: now also J7.36, U30.15, UE65.2
- net P6_A5: now also J7.38, U30.13, UE65.1
- net P6_CLK: now also J7.33, U30.18, UE64.1
- net P6_D0: now also J7.1, U28.18, UE60.1
- net P6_D1: now also J7.3, U28.17, UE60.2
- net P6_D10: now also J7.21, U29.16, UE62.4
- net P6_D11: now also J7.23, U29.15, UE62.5
- net P6_D12: now also J7.25, U29.14, UE63.1
- net P6_D13: now also J7.27, U29.13, UE63.2
- net P6_D14: now also J7.29, U29.12, UE63.4
- net P6_D15: now also J7.31, U29.11, UE63.5
- net P6_D2: now also J7.5, U28.16, UE60.4
- net P6_D3: now also J7.7, U28.15, UE60.5
- net P6_D4: now also J7.9, U28.14, UE61.1
- net P6_D5: now also J7.11, U28.13, UE61.2
- net P6_D6: now also J7.13, U28.12, UE61.4
- net P6_D7: now also J7.15, U28.11, UE61.5
- net P6_D8: now also J7.17, U29.18, UE62.1
- net P6_D9: now also J7.19, U29.17, UE62.2
- net P7_A0: now also J8.35, U33.16, UE74.2
- net P7_A1: now also J8.37, U33.14, UE74.4
- net P7_A2: now also J8.39, U33.12, UE74.5
- net P7_A3: now also J8.34, U33.17, UE75.4
- net P7_A4: now also J8.36, U33.15, UE75.2
- net P7_A5: now also J8.38, U33.13, UE75.1
- net P7_CLK: now also J8.33, U33.18, UE74.1
- net P7_D0: now also J8.1, U31.18, UE70.1
- net P7_D1: now also J8.3, U31.17, UE70.2
- net P7_D10: now also J8.21, U32.16, UE72.4
- net P7_D11: now also J8.23, U32.15, UE72.5
- net P7_D12: now also J8.25, U32.14, UE73.1
- net P7_D13: now also J8.27, U32.13, UE73.2
- net P7_D14: now also J8.29, U32.12, UE73.4
- net P7_D15: now also J8.31, U32.11, UE73.5
- net P7_D2: now also J8.5, U31.16, UE70.4
- net P7_D3: now also J8.7, U31.15, UE70.5
- net P7_D4: now also J8.9, U31.14, UE71.1
- net P7_D5: now also J8.11, U31.13, UE71.2
- net P7_D6: now also J8.13, U31.12, UE71.4
- net P7_D7: now also J8.15, U31.11, UE71.5
- net P7_D8: now also J8.17, U32.18, UE72.1
- net P7_D9: now also J8.19, U32.17, UE72.2
- net SW: now also C7.1, L1.1, U2.5
- net USB_DN: now also J9.A7, J9.B7, U1.13, U3.3, U3.4
- net USB_DP: now also J9.A6, J9.B6, U1.14, U3.1, U3.6
- net V12F: now also D3.2, D4.1, F1.2
- net VBUS: now also D1.2, J9.A4, J9.A9, J9.B4, J9.B9, U3.5
- net VIN: now also C1.1, C2.1, D1.1, D3.1, U2.2, U2.3
- net VIN12: now also F1.1, J10.1
- no-connect marks 16 -> 216
