File: hardware/main_v1/main_v1.kicad_pcb (KiCad board)
At the start: 2 copper layers, 300 x 130 mm, 90 parts, among them J1 PORT0, J10 12V_IN, J2 PORT1, J3 PORT2, J4 PORT3, J5 PORT4, J6 PORT5, J7 PORT6, J8 PORT7, J9 USB-C, SW1 BOOT, SW2 RESET, U1 ESP32-S3-WROOM-1-N16R8, U10 74LVC245APW, U11 74LVC245APW, U12 74LVC245APW, U13 74LVC245APW, U14 74LVC245APW, U15 74LVC245APW, U16 74LVC245APW, U17 74LVC245APW, U18 74LVC245APW, U19 74LVC245APW, U2 AP63203WU-7, U20 74LVC245APW, U21 74LVC245APW, U22 74LVC245APW, U23 74LVC245APW, U24 74LVC245APW, U25 74LVC245APW, U26 74LVC245APW, U27 74LVC245APW, U28 74LVC245APW, U29 74LVC245APW, U3 USBLC6-2SC6, U30 74LVC245APW, U31 74LVC245APW, U32 74LVC245APW, U33 74LVC245APW

Commit message: Size table + pixel choice, cube footprint lib (TPS25947 RPW, verified inductors), schematic->PCB linking (main parity 0), TPD4E05U06 port ESD, branch layout WIP
Parts:
- added UE0: TPD4E05U06DQAR, Package_SON:USON-10_2.5x1.0mm_P0.5mm, B.Cu at (61.8, 14.0)
- added UE1: TPD4E05U06DQAR, Package_SON:USON-10_2.5x1.0mm_P0.5mm, B.Cu at (72.0, 14.0)
- added UE10: TPD4E05U06DQAR, Package_SON:USON-10_2.5x1.0mm_P0.5mm, B.Cu at (121.8, 14.0)
- added UE11: TPD4E05U06DQAR, Package_SON:USON-10_2.5x1.0mm_P0.5mm, B.Cu at (132.0, 14.0)
- added UE12: TPD4E05U06DQAR, Package_SON:USON-10_2.5x1.0mm_P0.5mm, B.Cu at (142.1, 14.0)
- added UE13: TPD4E05U06DQAR, Package_SON:USON-10_2.5x1.0mm_P0.5mm, B.Cu at (152.3, 14.0)
- added UE14: TPD4E05U06DQAR, Package_SON:USON-10_2.5x1.0mm_P0.5mm, B.Cu at (162.4, 14.0)
- added UE15: TPD4E05U06DQAR, Package_SON:USON-10_2.5x1.0mm_P0.5mm, B.Cu at (161.2, 4.00)
- added UE2: TPD4E05U06DQAR, Package_SON:USON-10_2.5x1.0mm_P0.5mm, B.Cu at (82.1, 14.0)
- added UE20: TPD4E05U06DQAR, Package_SON:USON-10_2.5x1.0mm_P0.5mm, B.Cu at (181.8, 14.0)
- added UE21: TPD4E05U06DQAR, Package_SON:USON-10_2.5x1.0mm_P0.5mm, B.Cu at (192.0, 14.0)
- added UE22: TPD4E05U06DQAR, Package_SON:USON-10_2.5x1.0mm_P0.5mm, B.Cu at (202.1, 14.0)
- added UE23: TPD4E05U06DQAR, Package_SON:USON-10_2.5x1.0mm_P0.5mm, B.Cu at (212.3, 14.0)
- added UE24: TPD4E05U06DQAR, Package_SON:USON-10_2.5x1.0mm_P0.5mm, B.Cu at (222.4, 14.0)
- added UE25: TPD4E05U06DQAR, Package_SON:USON-10_2.5x1.0mm_P0.5mm, B.Cu at (221.2, 4.00)
- added UE3: TPD4E05U06DQAR, Package_SON:USON-10_2.5x1.0mm_P0.5mm, B.Cu at (92.3, 14.0)
- added UE30: TPD4E05U06DQAR, Package_SON:USON-10_2.5x1.0mm_P0.5mm, B.Cu at (241.8, 14.0)
- added UE31: TPD4E05U06DQAR, Package_SON:USON-10_2.5x1.0mm_P0.5mm, B.Cu at (252.0, 14.0)
- added UE32: TPD4E05U06DQAR, Package_SON:USON-10_2.5x1.0mm_P0.5mm, B.Cu at (262.1, 14.0)
- added UE33: TPD4E05U06DQAR, Package_SON:USON-10_2.5x1.0mm_P0.5mm, B.Cu at (272.3, 14.0)
- added UE34: TPD4E05U06DQAR, Package_SON:USON-10_2.5x1.0mm_P0.5mm, B.Cu at (282.4, 14.0)
- added UE35: TPD4E05U06DQAR, Package_SON:USON-10_2.5x1.0mm_P0.5mm, B.Cu at (281.2, 4.00)
- added UE4: TPD4E05U06DQAR, Package_SON:USON-10_2.5x1.0mm_P0.5mm, B.Cu at (102.5, 14.0)
- added UE40: TPD4E05U06DQAR, Package_SON:USON-10_2.5x1.0mm_P0.5mm, B.Cu at (100.0, 116.0)
- added UE41: TPD4E05U06DQAR, Package_SON:USON-10_2.5x1.0mm_P0.5mm, B.Cu at (89.8, 116.0)
- added UE42: TPD4E05U06DQAR, Package_SON:USON-10_2.5x1.0mm_P0.5mm, B.Cu at (79.6, 116.0)
- added UE43: TPD4E05U06DQAR, Package_SON:USON-10_2.5x1.0mm_P0.5mm, B.Cu at (69.5, 116.0)
- added UE44: TPD4E05U06DQAR, Package_SON:USON-10_2.5x1.0mm_P0.5mm, B.Cu at (59.3, 116.0)
- added UE45: TPD4E05U06DQAR, Package_SON:USON-10_2.5x1.0mm_P0.5mm, B.Cu at (60.6, 126.0)
- added UE5: TPD4E05U06DQAR, Package_SON:USON-10_2.5x1.0mm_P0.5mm, B.Cu at (101.2, 4.00)
- added UE50: TPD4E05U06DQAR, Package_SON:USON-10_2.5x1.0mm_P0.5mm, B.Cu at (159.9, 116.0)
- added UE51: TPD4E05U06DQAR, Package_SON:USON-10_2.5x1.0mm_P0.5mm, B.Cu at (149.8, 116.0)
- added UE52: TPD4E05U06DQAR, Package_SON:USON-10_2.5x1.0mm_P0.5mm, B.Cu at (139.6, 116.0)
- added UE53: TPD4E05U06DQAR, Package_SON:USON-10_2.5x1.0mm_P0.5mm, B.Cu at (129.5, 116.0)
- added UE54: TPD4E05U06DQAR, Package_SON:USON-10_2.5x1.0mm_P0.5mm, B.Cu at (119.3, 116.0)
- added UE55: TPD4E05U06DQAR, Package_SON:USON-10_2.5x1.0mm_P0.5mm, B.Cu at (120.6, 126.0)
- added UE60: TPD4E05U06DQAR, Package_SON:USON-10_2.5x1.0mm_P0.5mm, B.Cu at (219.9, 116.0)
- added UE61: TPD4E05U06DQAR, Package_SON:USON-10_2.5x1.0mm_P0.5mm, B.Cu at (209.8, 116.0)
- added UE62: TPD4E05U06DQAR, Package_SON:USON-10_2.5x1.0mm_P0.5mm, B.Cu at (199.6, 116.0)
- added UE63: TPD4E05U06DQAR, Package_SON:USON-10_2.5x1.0mm_P0.5mm, B.Cu at (189.5, 116.0)
- added UE64: TPD4E05U06DQAR, Package_SON:USON-10_2.5x1.0mm_P0.5mm, B.Cu at (179.3, 116.0)
- added UE65: TPD4E05U06DQAR, Package_SON:USON-10_2.5x1.0mm_P0.5mm, B.Cu at (180.6, 126.0)
- added UE70: TPD4E05U06DQAR, Package_SON:USON-10_2.5x1.0mm_P0.5mm, B.Cu at (279.9, 116.0)
- added UE71: TPD4E05U06DQAR, Package_SON:USON-10_2.5x1.0mm_P0.5mm, B.Cu at (269.8, 116.0)
- added UE72: TPD4E05U06DQAR, Package_SON:USON-10_2.5x1.0mm_P0.5mm, B.Cu at (259.6, 116.0)
- added UE73: TPD4E05U06DQAR, Package_SON:USON-10_2.5x1.0mm_P0.5mm, B.Cu at (249.5, 116.0)
- added UE74: TPD4E05U06DQAR, Package_SON:USON-10_2.5x1.0mm_P0.5mm, B.Cu at (239.3, 116.0)
- added UE75: TPD4E05U06DQAR, Package_SON:USON-10_2.5x1.0mm_P0.5mm, B.Cu at (240.6, 126.0)
- C1: footprint C_1206_3216Metric -> Capacitor_SMD:C_1206_3216Metric
- C10, C11, C12, C13, C14, C15, C16, C17, C18, C19, C2, C20, C21, C22, C23, C24, C25, C26, C27, C28, C29, C3, C30, C31, C32, C33, C4, C5, C6, C7: footprint C_0603_1608Metric -> Capacitor_SMD:C_0603_1608Metric
- C8: footprint C_1210_3225Metric -> Capacitor_SMD:C_1210_3225Metric
- D1, D3: footprint D_SMA -> Diode_SMD:D_SMA
- D2: footprint LED_0603_1608Metric -> LED_SMD:LED_0603_1608Metric
- D4: footprint D_SMB -> Diode_SMD:D_SMB
- F1: footprint Fuse_1812_4532Metric -> Fuse:Fuse_1812_4532Metric
- FID1, FID2, FID3: footprint Fiducial_1mm_Mask2mm -> Fiducial:Fiducial_1mm_Mask2mm
- H1, H2, H3, H4, H5: footprint MountingHole_3.2mm_M3 -> MountingHole:MountingHole_3.2mm_M3
- J1, J2, J3, J4, J5, J6, J7, J8: footprint IDC-Header_2x20_P2.54mm_Vertical -> Connector_IDC:IDC-Header_2x20_P2.54mm_Vertical
- J10: footprint TerminalBlock_Phoenix_MKDS-1,5-2-5.08_1x02_P5.08mm_Horizontal -> TerminalBlock_Phoenix:TerminalBlock_Phoenix_MKDS-1,5-2-5.08_1x02_P5.08mm_Horizontal
- J9: footprint USB_C_Receptacle_HRO_TYPE-C-31-M-12 -> Connector_USB:USB_C_Receptacle_HRO_TYPE-C-31-M-12
- L1: footprint L_Bourns_SRP7028A_7.3x6.6mm -> cube:L_Cjiang_FXL0630
- R1, R2, R3, R4, R5: footprint R_0603_1608Metric -> Resistor_SMD:R_0603_1608Metric
- SW1, SW2: footprint SW_Push_1P1T_XKB_TS-1187A -> Button_Switch_SMD:SW_Push_1P1T_XKB_TS-1187A
- U1: footprint ESP32-S3-WROOM-1 -> RF_Module:ESP32-S3-WROOM-1
- U10, U11, U12, U13, U14, U15, U16, U17, U18, U19, U20, U21, U22, U23, U24, U25, U26, U27, U28, U29, U30, U31, U32, U33: footprint TSSOP-20_4.4x6.5mm_P0.65mm -> Package_SO:TSSOP-20_4.4x6.5mm_P0.65mm
- U2: footprint TSOT-23-6 -> Package_TO_SOT_SMD:TSOT-23-6
- U3: footprint SOT-23-6 -> Package_TO_SOT_SMD:SOT-23-6
- moved C7 3.59 mm to (39.2, 99.5), turned to 90 degrees
Connections:
- net +3V3 renamed /+3V3
- net A0 renamed /A0
- net A1 renamed /A1
- net A2 renamed /A2
- net A3 renamed /A3
- net A4 renamed /A4
- net A5 renamed /A5
- net CC1 renamed /CC1
- net CC2 renamed /CC2
- net CLK renamed /CLK
- net D0 renamed /D0
- net D1 renamed /D1
- net D10 renamed /D10
- net D11 renamed /D11
- net D12 renamed /D12
- net D13 renamed /D13
- net D14 renamed /D14
- net D15 renamed /D15
- net D2 renamed /D2
- net D3 renamed /D3
- net D4 renamed /D4
- net D5 renamed /D5
- net D6 renamed /D6
- net D7 renamed /D7
- net D8 renamed /D8
- net D9 renamed /D9
- net EN renamed /EN
- net GND renamed /GND
- net IO0 renamed /IO0
- net LED renamed /LED
- net LED_K renamed /LED_K
- net OE_N renamed /OE_N
- net P0_A0 renamed /P0_A0
- net P0_A1 renamed /P0_A1
- net P0_A2 renamed /P0_A2
- net P0_A3 renamed /P0_A3
- net P0_A4 renamed /P0_A4
- net P0_A5 renamed /P0_A5
- net P0_CLK renamed /P0_CLK
- net P0_D0 renamed /P0_D0
- net P0_D1 renamed /P0_D1
- net P0_D10 renamed /P0_D10
- net P0_D11 renamed /P0_D11
- net P0_D12 renamed /P0_D12
- net P0_D13 renamed /P0_D13
- net P0_D14 renamed /P0_D14
- net P0_D15 renamed /P0_D15
- net P0_D2 renamed /P0_D2
- net P0_D3 renamed /P0_D3
- net P0_D4 renamed /P0_D4
- net P0_D5 renamed /P0_D5
- net P0_D6 renamed /P0_D6
- net P0_D7 renamed /P0_D7
- net P0_D8 renamed /P0_D8
- net P0_D9 renamed /P0_D9
- net P1_A0 renamed /P1_A0
- net P1_A1 renamed /P1_A1
- net P1_A2 renamed /P1_A2
- net P1_A3 renamed /P1_A3
- net P1_A4 renamed /P1_A4
- net P1_A5 renamed /P1_A5
- net P1_CLK renamed /P1_CLK
- net P1_D0 renamed /P1_D0
- net P1_D1 renamed /P1_D1
- net P1_D10 renamed /P1_D10
- net P1_D11 renamed /P1_D11
- net P1_D12 renamed /P1_D12
- net P1_D13 renamed /P1_D13
- net P1_D14 renamed /P1_D14
- net P1_D15 renamed /P1_D15
- net P1_D2 renamed /P1_D2
- net P1_D3 renamed /P1_D3
- net P1_D4 renamed /P1_D4
- net P1_D5 renamed /P1_D5
- net P1_D6 renamed /P1_D6
- net P1_D7 renamed /P1_D7
- net P1_D8 renamed /P1_D8
- net P1_D9 renamed /P1_D9
- net P2_A0 renamed /P2_A0
- net P2_A1 renamed /P2_A1
- net P2_A2 renamed /P2_A2
- net P2_A3 renamed /P2_A3
- net P2_A4 renamed /P2_A4
- net P2_A5 renamed /P2_A5
- net P2_CLK renamed /P2_CLK
- net P2_D0 renamed /P2_D0
- net P2_D1 renamed /P2_D1
- net P2_D10 renamed /P2_D10
- net P2_D11 renamed /P2_D11
- net P2_D12 renamed /P2_D12
- net P2_D13 renamed /P2_D13
- net P2_D14 renamed /P2_D14
- net P2_D15 renamed /P2_D15
- net P2_D2 renamed /P2_D2
- net P2_D3 renamed /P2_D3
- net P2_D4 renamed /P2_D4
- net P2_D5 renamed /P2_D5
- net P2_D6 renamed /P2_D6
- net P2_D7 renamed /P2_D7
- net P2_D8 renamed /P2_D8
- net P2_D9 renamed /P2_D9
- net P3_A0 renamed /P3_A0
- net P3_A1 renamed /P3_A1
- net P3_A2 renamed /P3_A2
- net P3_A3 renamed /P3_A3
- net P3_A4 renamed /P3_A4
- net P3_A5 renamed /P3_A5
- net P3_CLK renamed /P3_CLK
- net P3_D0 renamed /P3_D0
- net P3_D1 renamed /P3_D1
- net P3_D10 renamed /P3_D10
- net P3_D11 renamed /P3_D11
- net P3_D12 renamed /P3_D12
- net P3_D13 renamed /P3_D13
- net P3_D14 renamed /P3_D14
- net P3_D15 renamed /P3_D15
- net P3_D2 renamed /P3_D2
- net P3_D3 renamed /P3_D3
- net P3_D4 renamed /P3_D4
- net P3_D5 renamed /P3_D5
- net P3_D6 renamed /P3_D6
- net P3_D7 renamed /P3_D7
- net P3_D8 renamed /P3_D8
- net P3_D9 renamed /P3_D9
- net P4_A0 renamed /P4_A0
- net P4_A1 renamed /P4_A1
- net P4_A2 renamed /P4_A2
- net P4_A3 renamed /P4_A3
- net P4_A4 renamed /P4_A4
- net P4_A5 renamed /P4_A5
- net P4_CLK renamed /P4_CLK
- net P4_D0 renamed /P4_D0
- net P4_D1 renamed /P4_D1
- net P4_D10 renamed /P4_D10
- net P4_D11 renamed /P4_D11
- net P4_D12 renamed /P4_D12
- net P4_D13 renamed /P4_D13
- net P4_D14 renamed /P4_D14
- net P4_D15 renamed /P4_D15
- net P4_D2 renamed /P4_D2
- net P4_D3 renamed /P4_D3
- net P4_D4 renamed /P4_D4
- net P4_D5 renamed /P4_D5
- net P4_D6 renamed /P4_D6
- net P4_D7 renamed /P4_D7
- net P4_D8 renamed /P4_D8
- net P4_D9 renamed /P4_D9
- net P5_A0 renamed /P5_A0
- net P5_A1 renamed /P5_A1
- net P5_A2 renamed /P5_A2
- net P5_A3 renamed /P5_A3
- net P5_A4 renamed /P5_A4
- net P5_A5 renamed /P5_A5
- net P5_CLK renamed /P5_CLK
- net P5_D0 renamed /P5_D0
- net P5_D1 renamed /P5_D1
- net P5_D10 renamed /P5_D10
- net P5_D11 renamed /P5_D11
- net P5_D12 renamed /P5_D12
- net P5_D13 renamed /P5_D13
- net P5_D14 renamed /P5_D14
- net P5_D15 renamed /P5_D15
- net P5_D2 renamed /P5_D2
- net P5_D3 renamed /P5_D3
- net P5_D4 renamed /P5_D4
- net P5_D5 renamed /P5_D5
- net P5_D6 renamed /P5_D6
- net P5_D7 renamed /P5_D7
- net P5_D8 renamed /P5_D8
- net P5_D9 renamed /P5_D9
- net P6_A0 renamed /P6_A0
- net P6_A1 renamed /P6_A1
- net P6_A2 renamed /P6_A2
- net P6_A3 renamed /P6_A3
- net P6_A4 renamed /P6_A4
- net P6_A5 renamed /P6_A5
- net P6_CLK renamed /P6_CLK
- net P6_D0 renamed /P6_D0
- net P6_D1 renamed /P6_D1
- net P6_D10 renamed /P6_D10
- net P6_D11 renamed /P6_D11
- net P6_D12 renamed /P6_D12
- net P6_D13 renamed /P6_D13
- net P6_D14 renamed /P6_D14
- net P6_D15 renamed /P6_D15
- net P6_D2 renamed /P6_D2
- net P6_D3 renamed /P6_D3
- net P6_D4 renamed /P6_D4
- net P6_D5 renamed /P6_D5
- net P6_D6 renamed /P6_D6
- net P6_D7 renamed /P6_D7
- net P6_D8 renamed /P6_D8
- net P6_D9 renamed /P6_D9
- net P7_A0 renamed /P7_A0
- net P7_A1 renamed /P7_A1
- net P7_A2 renamed /P7_A2
- net P7_A3 renamed /P7_A3
- net P7_A4 renamed /P7_A4
- net P7_A5 renamed /P7_A5
- net P7_CLK renamed /P7_CLK
- net P7_D0 renamed /P7_D0
- net P7_D1 renamed /P7_D1
- net P7_D10 renamed /P7_D10
- net P7_D11 renamed /P7_D11
- net P7_D12 renamed /P7_D12
- net P7_D13 renamed /P7_D13
- net P7_D14 renamed /P7_D14
- net P7_D15 renamed /P7_D15
- net P7_D2 renamed /P7_D2
- net P7_D3 renamed /P7_D3
- net P7_D4 renamed /P7_D4
- net P7_D5 renamed /P7_D5
- net P7_D6 renamed /P7_D6
- net P7_D7 renamed /P7_D7
- net P7_D8 renamed /P7_D8
- net P7_D9 renamed /P7_D9
- net USB_DN renamed /USB_DN
- net USB_DP renamed /USB_DP
- net V12F renamed /V12F
- net VBUS renamed /VBUS
- net VIN renamed /VIN
- net VIN12 renamed /VIN12
- C7 pad 1: BST -> /SW
- C7 pad 2: SW -> /BST
- L1 pad 1: SW -> /SW
- U1 pad 15: (no net) -> unconnected-(U1-Pad15)
- U1 pad 16: (no net) -> unconnected-(U1-Pad16)
- U1 pad 26: (no net) -> unconnected-(U1-Pad26)
- U1 pad 28: (no net) -> unconnected-(U1-Pad28)
- U1 pad 29: (no net) -> unconnected-(U1-Pad29)
- U1 pad 30: (no net) -> unconnected-(U1-Pad30)
- U1 pad 36: (no net) -> unconnected-(U1-Pad36)
- U1 pad 37: (no net) -> unconnected-(U1-Pad37)
- U12 pad 11: (no net) -> unconnected-(U12-Pad11)
- U15 pad 11: (no net) -> unconnected-(U15-Pad11)
- U18 pad 11: (no net) -> unconnected-(U18-Pad11)
- U2 pad 5: SW -> /SW
- U2 pad 6: BST -> /BST
- U21 pad 11: (no net) -> unconnected-(U21-Pad11)
- U24 pad 11: (no net) -> unconnected-(U24-Pad11)
- U27 pad 11: (no net) -> unconnected-(U27-Pad11)
- U30 pad 11: (no net) -> unconnected-(U30-Pad11)
- U33 pad 11: (no net) -> unconnected-(U33-Pad11)
Routing:
- net /GND: track 96.4 -> 133.2 mm, vias 528 -> 529
- net SW: track 14.5 -> 0.00 mm, vias 2 -> 0
- net /EN: track 40.2 -> 52.1 mm
- net /SW: track 0.00 -> 8.30 mm
- net /VIN: track 46.0 -> 53.7 mm
- net /P2_CLK: track 13.3 -> 19.1 mm
- net /P1_CLK: track 13.3 -> 19.1 mm
- net /P6_D3: track 12.7 -> 18.5 mm
- net /P5_D3: track 12.7 -> 18.5 mm
- net /P1_D3: track 12.7 -> 18.5 mm
- net /P0_D8: track 18.3 -> 24.1 mm
- net /P0_D11: track 12.7 -> 18.5 mm
- net /P0_D12: track 11.8 -> 17.6 mm
- net /P0_A2: track 12.6 -> 18.4 mm
- net /P0_D3: track 12.7 -> 18.5 mm
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